File: cc2652p_ch340e/cc2652p_ch340e.brd (EAGLE design)
At the start: 25.3 x 57.3 mm, 35 parts, among them J3 CORTEX_DEBUG_SMD, J5 TYPE-C-31-M-12, Q1 SI2323DS, U1 MCP73831, U2 ap2112k-3.3, U3 XC61CN3202MR-G, U4 CH340E_MSOP10

Commit message: Add files via upload
Connections:
- net +5V: now also J1.1
- net GND: no longer J1.1
Routing:
- net +5V: track 54.9 -> 57.8 mm
Other:
- board text added: "5V"
Changed lines of the file:
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@@
 <text x="2.9" y="14.8" size="0.8128" layer="25" font="vector" ratio="12" rot="R90">TDI</text>
 <text x="2.9" y="12" size="0.8128" layer="25" font="vector" ratio="12" rot="R90">3V3</text>
-<text x="2.9" y="9.5" size="0.8128" layer="25" font="vector" ratio="12" rot="R90">GND</text>
+<text x="2.96" y="9.87" size="0.8128" layer="25" font="vector" ratio="12" rot="R90">5V</text>
 <text x="12.9" y="0.3" size="0.8128" layer="25" font="vector" ratio="12" rot="R90">PWR</text>
 <text x="1.8" y="52.2" size="0.8128" layer="25" font="vector" ratio="12">R</text>
@@
 <contactref element="U$1" pad="23"/>
 <contactref element="U$1" pad="19"/>
-<contactref element="J1" pad="1"/>
 <contactref element="J1" pad="7"/>
 <contactref element="J2" pad="1"/>
@@
 <wire x1="16.97" y1="12.38" x2="17.05" y2="12.3" width="0.508" layer="1"/>
 <wire x1="16.3" y1="14" x2="16.97" y2="13.33" width="0.508" layer="1"/>
-<wire x1="3.49" y1="9.678" x2="3.54" y2="9.628" width="0.2" layer="1"/>
-<wire x1="3.54" y1="9.628" x2="3.54" y2="9.16" width="0.2" layer="1"/>
-<wire x1="3.54" y1="9.16" x2="4" y2="8.7" width="0.2" layer="1"/>
-<wire x1="4" y1="8.7" x2="4" y2="7.845" width="0.2" layer="1"/>
+<wire x1="3.49" y1="9.678" x2="3.5" y2="9.668" width="0.2" layer="1"/>
 <contactref element="R14" pad="2"/>
 <wire x1="17.25" y1="14.458" x2="16.352" y2="14.458" width="0.2" layer="1"/>
@@
 <wire x1="8.85" y1="10.4" x2="8.85" y2="9.41" width="0.4064" layer="1"/>
 <wire x1="12.3" y1="7.332" x2="13.9" y2="7.332" width="0.2" layer="1"/>
+<contactref element="J1" pad="1"/>
+<wire x1="3.95" y1="7.795" x2="3.95" y2="8.73" width="0.4064" layer="1"/>
+<wire x1="3.5" y1="9.18" x2="3.5" y2="9.668" width="0.4064" layer="1"/>
+<wire x1="3.95" y1="8.73" x2="3.5" y2="9.18" width="0.4064" layer="1"/>
+<wire x1="3.49" y1="9.678" x2="1.922" y2="9.678" width="0.4064" layer="1"/>
+<wire x1="1.922" y1="9.678" x2="1" y2="10.6" width="0.4064" layer="1"/>
 </signal>
 <signal name="UVCC">

Commit message: Add files via upload
Connections:
- net +5V: now also U4.10
Routing:
- net +5V: track 57.8 -> 59.1 mm
Changed lines of the file:
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@@
 <drawing>
 <settings>
-<setting alwaysvectorfont="yes"/>
+<setting alwaysvectorfont="no"/>
 <setting verticaltext="up"/>
 </settings>
@@
 <wire x1="8.85" y1="10.4" x2="8.85" y2="9.65" width="0.3048" layer="1"/>
 <wire x1="8.85" y1="9.65" x2="8.83" y2="9.63" width="0.3048" layer="1"/>
-<wire x1="11.34289375" y1="10.4" x2="8.85" y2="10.4" width="0.4064" layer="1"/>
+<wire x1="11.34289375" y1="10.4" x2="10.31" y2="10.4" width="0.4064" layer="1"/>
+<wire x1="10.31" y1="10.4" x2="8.85" y2="10.4" width="0.4064" layer="1"/>
 <wire x1="12.14289375" y1="11.2" x2="11.34289375" y2="10.4" width="0.4064" layer="1"/>
 <wire x1="8.85" y1="10.4" x2="8.85" y2="9.41" width="0.4064" layer="1"/>
@@
 <wire x1="3.49" y1="9.678" x2="1.922" y2="9.678" width="0.4064" layer="1"/>
 <wire x1="1.922" y1="9.678" x2="1" y2="10.6" width="0.4064" layer="1"/>
+<contactref element="U4" pad="10"/>
+<wire x1="10.35" y1="11.69" x2="10.35" y2="10.44" width="0.2" layer="1"/>
+<wire x1="10.35" y1="10.44" x2="10.31" y2="10.4" width="0.2" layer="1"/>
 </signal>
 <signal name="UVCC">

Commit message: Add files via upload
Connections:
- net +3V3: now also R9.1, U4.10, U4.7
- net +5V: no longer R9.1, U4.10, U4.7
Routing:
- net +3V3: track 61.7 -> 76.5 mm, vias 4 -> 6
- net +5V: track 59.1 -> 53.6 mm
- net GND: vias 140 -> 139
Changed lines of the file:
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@@
 <drawing>
 <settings>
-<setting alwaysvectorfont="no"/>
+<setting alwaysvectorfont="yes"/>
 <setting verticaltext="up"/>
 </settings>
-<grid distance="0.01" unitdist="mm" unit="mm" style="lines" multiple="1" display="yes" altdistance="0.1" altunitdist="mm" altunit="mm"/>
+<grid distance="0.127" unitdist="mm" unit="mm" style="lines" multiple="1" display="yes" altdistance="0.1" altunitdist="mm" altunit="mm"/>
 <layers>
 <layer number="1" name="Top" color="4" fill="1" visible="yes" active="yes"/>
@@
 <via x="14.61" y="9.73" extent="1-16" drill="0.3"/>
 <via x="7.03" y="9.43" extent="1-16" drill="0.3"/>
-<via x="12.09" y="14.57" extent="1-16" drill="0.3"/>
 <via x="13.42" y="13.42" extent="1-16" drill="0.3"/>
-<via x="12.08" y="12.47" extent="1-16" drill="0.3"/>
-<via x="11.86" y="16.12" extent="1-16" drill="0.3"/>
 <via x="6.6" y="18.71" extent="1-16" drill="0.3"/>
 <via x="7.28" y="14.35" extent="1-16" drill="0.3"/>
+<via x="12.184" y="14.976" extent="1-16" drill="0.3"/>
+<via x="12.15" y="12.531" extent="1-16" drill="0.3"/>
 </signal>
 <signal name="RESET">
@@
 <wire x1="17.25" y1="14.458" x2="16.352" y2="14.458" width="0.2" layer="1"/>
 <wire x1="16.352" y1="14.458" x2="16.3" y2="14.51" width="0.2" layer="1"/>
-<contactref element="U4" pad="7"/>
-<contactref element="R9" pad="1"/>
 <wire x1="8.83" y1="9.41" x2="8.85" y2="9.43" width="0.254" layer="1"/>
 <wire x1="8.83" y1="9.63" x2="8.83" y2="9.41" width="0.4064" layer="1"/>
 <wire x1="16.8" y1="11.2" x2="12.14289375" y2="11.2" width="0.4064" layer="1"/>
-<wire x1="8.83" y1="9.41" x2="13.68" y2="9.41" width="0.2" layer="16"/>
-<wire x1="13.68" y1="9.41" x2="14.83" y2="8.26" width="0.2" layer="16"/>
-<wire x1="14.83" y1="8.26" x2="14.83" y2="7.33" width="0.2" layer="16"/>
-<wire x1="14.83" y1="7.33" x2="14.8" y2="7.3" width="0.2" layer="16"/>
-<wire x1="8.85" y1="11.69" x2="8.85" y2="10.4" width="0.3048" layer="1"/>
-<wire x1="8.85" y1="10.4" x2="8.85" y2="9.65" width="0.3048" layer="1"/>
 <wire x1="8.85" y1="9.65" x2="8.83" y2="9.63" width="0.3048" layer="1"/>
-<wire x1="11.34289375" y1="10.4" x2="10.31" y2="10.4" width="0.4064" layer="1"/>
-<wire x1="10.31" y1="10.4" x2="8.85" y2="10.4" width="0.4064" layer="1"/>
 <wire x1="12.14289375" y1="11.2" x2="11.34289375" y2="10.4" width="0.4064" layer="1"/>
-<wire x1="8.85" y1="10.4" x2="8.85" y2="9.41" width="0.4064" layer="1"/>
-<wire x1="12.3" y1="7.332" x2="13.9" y2="7.332" width="0.2" layer="1"/>
 <contactref element="J1" pad="1"/>
 <wire x1="3.95" y1="7.795" x2="3.95" y2="8.73" width="0.4064" layer="1"/>
@@
 <wire x1="3.49" y1="9.678" x2="1.922" y2="9.678" width="0.4064" layer="1"/>
 <wire x1="1.922" y1="9.678" x2="1" y2="10.6" width="0.4064" layer="1"/>
-<contactref element="U4" pad="10"/>
-<wire x1="10.35" y1="11.69" x2="10.35" y2="10.44" width="0.2" layer="1"/>
-<wire x1="10.35" y1="10.44" x2="10.31" y2="10.4" width="0.2" layer="1"/>
+<wire x1="14.8" y1="7.3" x2="12.131" y2="7.3" width="0.2" layer="16"/>
+<wire x1="12.131" y1="7.3" x2="11.684" y2="7.747" width="0.2" layer="16"/>
+<wire x1="11.684" y1="7.747" x2="11.684" y2="9.017" width="0.2" layer="16"/>
+<wire x1="11.684" y1="9.017" x2="11.291" y2="9.41" width="0.2" layer="16"/>
+<wire x1="11.291" y1="9.41" x2="8.83" y2="9.41" width="0.2" layer="16"/>
+<wire x1="11.34289375" y1="10.4" x2="9.6" y2="10.4" width="0.4064" layer="1"/>
+<wire x1="9.6" y1="10.4" x2="8.85" y2="9.65" width="0.4064" layer="1"/>
 </signal>
 <signal name="UVCC">
@@
 <wire x1="9.168" y1="17.368" x2="9.1" y2="17.3" width="0.2" layer="1"/>
 <via x="9.1" y="17.3" extent="1-16" drill="0.3"/>
-<wire x1="9.1" y1="17.3" x2="9.1" y2="18.9952" width="0.2" layer="16"/>
-<wire x1="9.1" y1="18.9952" x2="9.4" y2="19.2952" width="0.2" layer="16"/>
-<wire x1="9.4" y1="19.2952" x2="10.69195" y2="19.2952" width="0.2" layer="16"/>
-<wire x1="11.59675" y1="20.2" x2="17.1" y2="20.2" width="0.2" layer="16"/>
-<wire x1="10.69195" y1="19.2952" x2="11.59675" y2="20.2" width="0.2" layer="16"/>
 <via x="6.9" y="21.3" extent="1-16" drill="0.3"/>
 <wire x1="4.327" y1="24.9" x2="4.287" y2="24.94" width="0.2" layer="1"/>
@@
 <wire x1="4.7158" y1="29.84910625" x2="4.7158" y2="26.9458" width="0.254" layer="1"/>
 <wire x1="4.7158" y1="26.9458" x2="4.287" y2="26.517" width="0.254" layer="1"/>
+<contactref element="U4" pad="7"/>
+<contactref element="R9" pad="1"/>
+<contactref element="U4" pad="10"/>
+<wire x1="9.1" y1="17.3" x2="9.1" y2="18.8728" width="0.3048" layer="16"/>
+<wire x1="9.1" y1="18.8728" x2="9.47" y2="19.2428" width="0.3048" layer="16"/>
+<wire x1="9.47" y1="19.2428" x2="10.71365" y2="19.2428" width="0.3048" layer="16"/>
+<wire x1="11.67085" y1="20.2" x2="17.1" y2="20.2" width="0.3048" layer="16"/>
+<wire x1="10.71365" y1="19.2428" x2="11.67085" y2="20.2" width="0.3048" layer="16"/>
+<wire x1="12.3" y1="7.332" x2="12.3" y2="8.109" width="0.2" layer="1"/>
+<wire x1="12.3" y1="8.109" x2="12.319" y2="8.128" width="0.2" layer="1"/>
+<via x="12.319" y="8.128" extent="1-16" drill="0.3"/>
+<wire x1="8.85" y1="11.69" x2="8.85" y2="11.0226" width="0.2" layer="1"/>
+<wire x1="8.85" y1="11.0226" x2="9.017" y2="10.8556" width="0.2" layer="1"/>
+<wire x1="9.017" y1="10.8556" x2="10.16" y2="10.8556" width="0.2" layer="1"/>
+<wire x1="10.16" y1="10.8556" x2="10.35" y2="11.0456" width="0.2" layer="1"/>
+<wire x1="10.35" y1="11.0456" x2="10.35" y2="11.69" width="0.2" layer="1"/>
+<wire x1="10.3" y1="17.368" x2="11.303" y2="16.365" width="0.2" layer="1"/>
+<wire x1="11.049" y1="11.684" x2="10.356" y2="11.684" width="0.2" layer="1"/>
+<wire x1="10.356" y1="11.684" x2="10.35" y2="11.69" width="0.2" layer="1"/>
+<wire x1="11.303" y1="16.365" x2="11.303" y2="11.938" width="0.2" layer="1"/>
+<via x="11.303" y="11.938" extent="1-16" drill="0.3"/>
+<wire x1="11.303" y1="11.938" x2="11.049" y2="11.684" width="0.2" layer="1"/>
+<wire x1="12.319" y1="8.128" x2="12.319" y2="10.922" width="0.2" layer="16"/>
+<wire x1="12.319" y1="10.922" x2="11.303" y2="11.938" width="0.2" layer="16"/>
 </signal>
 <signal name="CC2">
