File: cc2652p_ch340e/cc2652p_ch340e.brd (EAGLE design)
At the start: 25.3 x 57.3 mm, 35 parts, among them J3 CORTEX_DEBUG_SMD, J5 TYPE-C-31-M-12, Q1 SI2323DS, U1 MCP73831, U2 ap2112k-3.3, U3 XC61CN3202MR-G, U4 CH340E_MSOP10

Commit message: Add files via upload
Parts:
- removed C3: 0.1uF, SparkFun-Capacitors:0603
- removed CN1: (no value), adafruit:JST-PH-2-SMT-RA
- removed R1: 100k, RC0402FR-073M6L:RESC1005X40N
- added C13: 220uF, Capacitor:CAPM7343X310
- added C4: 100n, discretes-dev:CAPC1005X40N
- added CN2: (no value), adafruit:JST-PH-2-SMT-RA
- added PAD1, PAD2: WIREPADSMD1,27-254, wirepad:SMD1,27-2,54
- added Q2: SI2323DS, SI2323DS:SOT23
- added R15, R16: 0, RC0402FR-073M6L:RESC1005X40N
- added R17, R18: 100k, RC0402FR-073M6L:RESC1005X40N
- added R6: 2.2k, RC0402FR-073M6L:RESC1005X40N
- added SJ1: PSM, pimoroni-misc:SMALL_SOLDER_JUMPER_CLOSED
- added U$2: MX25R8035FM1IL0, W25Q80BVSNIG:SO-8
- added U5: MMDT2907A-7-F, MMDT2907A-7-F:SOT65P210X110-6N
- added U6: MX25R8035FZUIL0, MX25R8035FZUIL0:PSON50P200X300X60-9N
- D5: value (none) -> MBR0540
- moved Q1 0.10 mm to (16.0, 11.2)
- moved D5 0.10 mm to (15.0, 15.3)
Connections:
- new net N$10: Q2.1, R17.2, U5.6
- new net N$12: R15.2, U$2.7, U6.7
- new net N$15: R16.1, U$2.3, U6.3
- new net N$4: R18.2, U5.2, U5.3, U5.5
- new net V+: C2.1, Q2.3, R9.1, SJ1.1, U2.5, U4.10, U4.7, U5.4
- net +3V3: now also C13.1, C4.2, Q2.2, R15.1, R16.2, R6.1, SJ1.2, U$2.8, U5.1, U6.8; no longer C2.1, R1.1, R9.1, U2.5, U4.10, U4.7
- net DIO_10: now also U$2.6, U6.6
- net DIO_20: now also R6.2, U$2.1, U6.1
- net DIO_8: now also U$2.2, U6.2
- net DIO_9: now also U$2.5, U6.5
- net GND: now also C13.2, C4.1, CN2.2, J5.S5, J5.S6, PAD1.1, R17.1, R18.1, U$2.4, U6.4, U6.9; no longer C3.2, CN1.2, J5.S1, J5.S2
- net RESET: no longer C3.1, R1.2
- net VCC: now also CN2.1, PAD2.1; no longer CN1.1
Routing:
- net V+: track 0.00 -> 43.6 mm, vias 0 -> 2
- net DIO_20: track 13.2 -> 40.2 mm, vias 0 -> 1
- net DIO_8: track 18.0 -> 36.9 mm, vias 2 -> 3
- net +3V3: track 76.5 -> 91.0 mm, vias 6 -> 2
- net DIO_10: track 3.09 -> 14.4 mm, vias 0 -> 1
- net DIO_9: track 3.97 -> 13.4 mm, vias 0 -> 1
- net N$12: track 0.00 -> 8.55 mm
- net N$10: track 0.00 -> 7.16 mm
- net N$15: track 0.00 -> 6.86 mm
- net N$4: track 0.00 -> 4.46 mm
- net VCC: track 48.8 -> 52.9 mm, vias 8 -> 10
- net GND: track 17.9 -> 15.8 mm, vias 139 -> 76
- net DIO_14: track 37.8 -> 36.4 mm
- net DIO_7: track 31.8 -> 30.5 mm
Other:
- outline, holes or cut-outs redrawn
- board text added: "+"
- board text added: "-"
- board text added: "DIO12/RX"
- board text added: "DIO13/TX"
- board text added: "TDI/DIO17"
- board text added: "TDO/DIO16"
- board text removed: "DIO12"
- board text removed: "DIO13"
