File: cc2652p_ch340e/cc2652p_ch340e.sch (EAGLE design)
At the start: 35 parts, among them J3 CORTEX_DEBUG_SMD, J5 TYPE-C-31-M-12, Q1 SI2323DS, U1 MCP73831, U2 ap2112k-3.3, U3 XC61CN3202MR-G, U4 CH340E_MSOP10

Commit message: Add files via upload
Connections:
- net +5V: now also J1.1
- net GND: no longer J1.1
Changed lines of the file:
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@@
 <part name="U4" library="CH340E" deviceset="CH340E" device="_MSOP10"/>
 <part name="GND11" library="supply1" library_urn="urn:adsk.eagle:library:371" deviceset="GND" device=""/>
+<part name="P+6" library="supply1" library_urn="urn:adsk.eagle:library:371" deviceset="+5V" device=""/>
 </parts>
 <sheets>
@@
 <attribute name="VALUE" x="30.48" y="116.84" size="1.778" layer="96"/>
 </instance>
+<instance part="P+6" gate="1" x="104.14" y="55.88" smashed="yes" rot="R270">
+<attribute name="VALUE" x="96.52" y="55.88" size="1.778" layer="96"/>
+</instance>
 </instances>
 <busses>
@@
 <wire x1="43.18" y1="33.02" x2="43.18" y2="25.4" width="0.1524" layer="91"/>
 <pinref part="GND22" gate="1" pin="GND"/>
-</segment>
-<segment>
-<pinref part="J1" gate="G$1" pin="1"/>
-<wire x1="93.98" y1="55.88" x2="101.6" y2="55.88" width="0.1524" layer="91"/>
-<label x="96.52" y="55.88" size="1.778" layer="95"/>
 </segment>
 <segment>
@@
 <junction x="30.48" y="142.24"/>
 </segment>
-</net>
+<segment>
+<pinref part="J1" gate="G$1" pin="1"/>
+<pinref part="P+6" gate="1" pin="+5V"/>
+<wire x1="93.98" y1="55.88" x2="101.6" y2="55.88" width="0.1524" layer="91"/>
+</segment>
+</net>

Commit message: Add files via upload
Connections:
- net +5V: now also U4.V3
Changed lines of the file:
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@@
 <wire x1="30.48" y1="152.4" x2="30.48" y2="142.24" width="0.1524" layer="91"/>
 <junction x="30.48" y="142.24"/>
+<pinref part="U4" gate="U1" pin="V3"/>
+<wire x1="38.1" y1="139.7" x2="30.48" y2="139.7" width="0.1524" layer="91"/>
+<wire x1="30.48" y1="139.7" x2="30.48" y2="142.24" width="0.1524" layer="91"/>
 </segment>
 <segment>

Commit message: Add files via upload
Connections:
- net +3V3: now also R9.1, U4.V3, U4.VCC
- net +5V: no longer R9.1, U4.V3, U4.VCC
Changed lines of the file:
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@@
 <part name="R12" library="RC0402FR-073M6L" deviceset="RC0402FR-073M6L" device="" value="2.2k"/>
 <part name="D6" library="SparkFun-LED" library_urn="urn:adsk.eagle:library:529" deviceset="LED-BLUE" device="0603" package3d_urn="urn:adsk.eagle:package:39354/1" value="BLUE"/>
-<part name="P+5" library="supply1" library_urn="urn:adsk.eagle:library:371" deviceset="+5V" device=""/>
 <part name="J3" library="SparkFun-Connectors" library_urn="urn:adsk.eagle:library:513" deviceset="CORTEX_DEBUG" device="_SMD" package3d_urn="urn:adsk.eagle:package:38289/1"/>
 <part name="GND20" library="supply1" library_urn="urn:adsk.eagle:library:371" deviceset="GND" device=""/>
@@
 <part name="GND11" library="supply1" library_urn="urn:adsk.eagle:library:371" deviceset="GND" device=""/>
 <part name="P+6" library="supply1" library_urn="urn:adsk.eagle:library:371" deviceset="+5V" device=""/>
+<part name="+3V3" library="supply1" library_urn="urn:adsk.eagle:library:371" deviceset="+3V3" device=""/>
 </parts>
 <sheets>
 <sheet>
 <plain>
+<wire x1="96.52" y1="147.32" x2="121.92" y2="127" width="0.508" layer="94"/>
+<wire x1="96.52" y1="127" x2="121.92" y2="147.32" width="0.508" layer="94"/>
 </plain>
 <instances>
@@
 <attribute name="VALUE" x="191.135" y="182.372" size="1.778" layer="96" font="vector" rot="R270" align="top-left"/>
 </instance>
-<instance part="P+5" gate="1" x="30.48" y="154.94" smashed="yes">
-<attribute name="VALUE" x="27.94" y="149.86" size="1.778" layer="96" rot="R90"/>
-</instance>
 <instance part="J3" gate="G$1" x="165.1" y="58.42" smashed="yes">
 <attribute name="NAME" x="152.4" y="66.294" size="1.778" layer="95" font="vector"/>
@@
 <instance part="P+6" gate="1" x="104.14" y="55.88" smashed="yes" rot="R270">
 <attribute name="VALUE" x="96.52" y="55.88" size="1.778" layer="96"/>
+</instance>
+<instance part="+3V3" gate="G$1" x="30.48" y="149.86" smashed="yes">
+<attribute name="VALUE" x="27.94" y="144.78" size="1.778" layer="96" rot="R90"/>
 </instance>
 </instances>
@@
 </segment>
 <segment>
-<pinref part="U4" gate="U1" pin="VCC"/>
-<pinref part="R9" gate="G$1" pin="1"/>
-<wire x1="38.1" y1="142.24" x2="30.48" y2="142.24" width="0.1524" layer="91"/>
-<pinref part="P+5" gate="1" pin="+5V"/>
-<wire x1="30.48" y1="142.24" x2="25.4" y2="142.24" width="0.1524" layer="91"/>
-<wire x1="30.48" y1="152.4" x2="30.48" y2="142.24" width="0.1524" layer="91"/>
-<junction x="30.48" y="142.24"/>
-<pinref part="U4" gate="U1" pin="V3"/>
-<wire x1="38.1" y1="139.7" x2="30.48" y2="139.7" width="0.1524" layer="91"/>
-<wire x1="30.48" y1="139.7" x2="30.48" y2="142.24" width="0.1524" layer="91"/>
-</segment>
-<segment>
 <pinref part="J1" gate="G$1" pin="1"/>
 <pinref part="P+6" gate="1" pin="+5V"/>
@@
 <pinref part="+3V4" gate="G$1" pin="+3V3"/>
 </segment>
-</net>
+<segment>
+<pinref part="U4" gate="U1" pin="VCC"/>
+<pinref part="R9" gate="G$1" pin="1"/>
+<wire x1="38.1" y1="142.24" x2="30.48" y2="142.24" width="0.1524" layer="91"/>
+<wire x1="30.48" y1="142.24" x2="25.4" y2="142.24" width="0.1524" layer="91"/>
+<junction x="30.48" y="142.24"/>
+<pinref part="U4" gate="U1" pin="V3"/>
+<wire x1="38.1" y1="139.7" x2="30.48" y2="139.7" width="0.1524" layer="91"/>
+<wire x1="30.48" y1="139.7" x2="30.48" y2="142.24" width="0.1524" layer="91"/>
+<pinref part="+3V3" gate="G$1" pin="+3V3"/>
+<wire x1="30.48" y1="142.24" x2="30.48" y2="147.32" width="0.1524" layer="91"/>
+</segment>
+</net>

Commit message: Add files via upload
Parts:
- removed C3: 0.1uF, SparkFun-Capacitors:0.1UF-0603-25V-(+80/-20%)
- removed CN1: (no value), adafruit:JST_2PIN-SMT-RA
- removed R1: 100k, RC0402FR-073M6L:RC0402FR-073M6L
- added C13: 220uF, Capacitor:C_TANTALUM-2917(7343-METRIC)
- added C4: 100n, discretes-dev:CAP0402
- added CN2: (no value), adafruit:JST_2PIN-SMT-RA
- added PAD1, PAD2: WIREPADSMD1,27-254, wirepad:WIREPADSMD1,27-254
- added Q2: SI2323DS, SI2323DS:SI2323DS
- added R15, R16: 0, RC0402FR-073M6L:RC0402FR-073M6L
- added R17, R18: 100k, RC0402FR-073M6L:RC0402FR-073M6L
- added R6: 2.2k, RC0402FR-073M6L:RC0402FR-073M6L
- added SJ1: PSM, pimoroni-misc:SMALL_SOLDER_JUMPER_CLOSED
- added U$2: MX25R8035FM1IL0, W25Q80BVSNIG:W25Q80BVSNIG
- added U5: MMDT2907A-7-F, MMDT2907A-7-F:MMDT2907A-7-F
- added U6: MX25R8035FZUIL0, MX25R8035FZUIL0:MX25R8035FZUIL0
- D5: value (none) -> MBR0540
Connections:
- new net N$10: Q2.G, R17.2, U5.C2
- new net N$12: R15.2, U$2.HOLD/IO3, U6.!RESET!/SIO3
- new net N$15: R16.1, U$2.WP/IO2, U6.!WP!/SIO2
- new net N$4: R18.2, U5.B1, U5.B2, U5.C1
- new net V+: C2.1, Q2.D, R9.1, SJ1.1, U2.OUT, U4.V3, U4.VCC, U5.E1
- net +3V3: now also C13.1, C4.2, Q2.S, R15.1, R16.2, R6.1, SJ1.2, U$2.VCC, U5.E2, U6.VCC; no longer C2.1, R1.1, R9.1, U2.OUT, U4.V3, U4.VCC
- net DIO_10: now also U$2.CLK, U6.SCLK
- net DIO_20: now also R6.2, U$2.CS, U6.!CS
- net DIO_8: now also U$2.DO/IO1, U6.SO/SIO1
- net DIO_9: now also U$2.DI/IO0, U6.SI/SIO0
- net GND: now also C13.2, C4.1, CN2.1, PAD1.P, R17.1, R18.1, U$2.GND, U6.EXP, U6.GND; no longer C3.2, CN1.1
- net RESET: no longer C3.1, R1.2
- net VCC: now also CN2.2, PAD2.P; no longer CN1.2
Other:
- moved on the sheet: D6, R11, R12, R2, U1, U3
