File: cc2652p_ch340k/cc2652p_ch340k.brd (EAGLE design)
At the start: 25.3 x 57.3 mm, 35 parts, among them J3 CORTEX_DEBUG_SMD, J5 TYPE-C-31-M-12, Q1 SI2323DS, U1 MCP73831, U2 ap2112k-3.3, U3 XC61CN3202MR-G

Commit message: Add files via upload
Connections:
- net +5V: now also J1.1
- net GND: no longer J1.1
Routing:
- net +5V: track 55.0 -> 57.9 mm
Other:
- board text added: "5V"
Changed lines of the file:
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@@
 <drawing>
 <settings>
-<setting alwaysvectorfont="yes"/>
+<setting alwaysvectorfont="no"/>
 <setting verticaltext="up"/>
 </settings>
@@
 <text x="2.9" y="14.8" size="0.8128" layer="25" font="vector" ratio="12" rot="R90">TDI</text>
 <text x="2.9" y="12" size="0.8128" layer="25" font="vector" ratio="12" rot="R90">3V3</text>
-<text x="2.9" y="9.5" size="0.8128" layer="25" font="vector" ratio="12" rot="R90">GND</text>
+<text x="2.9" y="9.881" size="0.8128" layer="25" font="vector" ratio="12" rot="R90">5V</text>
 <text x="12.9" y="0.3" size="0.8128" layer="25" font="vector" ratio="12" rot="R90">PWR</text>
 <text x="1.8" y="52.2" size="0.8128" layer="25" font="vector" ratio="12">R</text>
@@
 <contactref element="U$1" pad="23"/>
 <contactref element="U$1" pad="19"/>
-<contactref element="J1" pad="1"/>
 <contactref element="J1" pad="7"/>
 <contactref element="J2" pad="1"/>
@@
 <wire x1="16.97" y1="12.38" x2="17.05" y2="12.3" width="0.508" layer="1"/>
 <wire x1="16.3" y1="14" x2="16.97" y2="13.33" width="0.508" layer="1"/>
-<wire x1="3.49" y1="9.678" x2="3.54" y2="9.628" width="0.2" layer="1"/>
-<wire x1="3.54" y1="9.628" x2="3.54" y2="9.16" width="0.2" layer="1"/>
-<wire x1="3.54" y1="9.16" x2="4" y2="8.7" width="0.2" layer="1"/>
-<wire x1="4" y1="8.7" x2="4" y2="7.845" width="0.2" layer="1"/>
+<wire x1="3.54" y1="9.628" x2="3.49" y2="9.678" width="0.2" layer="1"/>
 <contactref element="R14" pad="2"/>
 <wire x1="17.25" y1="14.458" x2="16.352" y2="14.458" width="0.2" layer="1"/>
@@
 <wire x1="9.414" y1="10.869" x2="9.414" y2="9.172" width="0.4064" layer="1"/>
 <wire x1="9.414" y1="9.172" x2="9.271" y2="9.029" width="0.4064" layer="1"/>
+<contactref element="J1" pad="1"/>
+<wire x1="3.95" y1="7.795" x2="3.95" y2="8.75" width="0.4064" layer="1"/>
+<wire x1="3.54" y1="9.16" x2="3.54" y2="9.628" width="0.4064" layer="1"/>
+<wire x1="3.95" y1="8.75" x2="3.54" y2="9.16" width="0.4064" layer="1"/>
+<wire x1="3.49" y1="9.678" x2="1.922" y2="9.678" width="0.4064" layer="1"/>
+<wire x1="1.922" y1="9.678" x2="1" y2="10.6" width="0.4064" layer="1"/>
 </signal>
 <signal name="UVCC">

Commit message: Add files via upload
Parts:
- moved U$2 0.63 mm to (10.7, 14.0)
Connections:
- net +3V3: now also U$2.P$6, U$2.P$9
- net +5V: no longer U$2.P$6
Routing:
- net +3V3: track 60.4 -> 77.5 mm, vias 4 -> 5
- net +5V: track 57.9 -> 56.0 mm
- net DIO_12: track 42.9 -> 42.2 mm
- net RTS: track 14.1 -> 13.6 mm
