File: cc2652p_ch340k/cc2652p_ch340k.sch (EAGLE design)
At the start: 35 parts, among them J3 CORTEX_DEBUG_SMD, J5 TYPE-C-31-M-12, Q1 SI2323DS, U1 MCP73831, U2 ap2112k-3.3, U3 XC61CN3202MR-G

Commit message: Add files via upload
Connections:
- net +5V: now also J1.1
- net GND: no longer J1.1
Changed lines of the file:
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@@
 <part name="U$2" library="CH340" deviceset="CH340K" device=""/>
 <part name="P+6" library="supply1" library_urn="urn:adsk.eagle:library:371" deviceset="+5V" device=""/>
+<part name="P+8" library="supply1" library_urn="urn:adsk.eagle:library:371" deviceset="+5V" device=""/>
 </parts>
 <sheets>
@@
 <attribute name="VALUE" x="78.74" y="119.38" size="1.778" layer="96"/>
 </instance>
+<instance part="P+8" gate="1" x="104.14" y="55.88" smashed="yes" rot="R270">
+<attribute name="VALUE" x="96.52" y="55.88" size="1.778" layer="96"/>
+</instance>
 </instances>
 <busses>
@@
 <wire x1="43.18" y1="33.02" x2="43.18" y2="25.4" width="0.1524" layer="91"/>
 <pinref part="GND22" gate="1" pin="GND"/>
-</segment>
-<segment>
-<pinref part="J1" gate="G$1" pin="1"/>
-<wire x1="93.98" y1="55.88" x2="101.6" y2="55.88" width="0.1524" layer="91"/>
-<label x="96.52" y="55.88" size="1.778" layer="95"/>
 </segment>
 <segment>
@@
 <pinref part="P+6" gate="1" pin="+5V"/>
 </segment>
-</net>
+<segment>
+<pinref part="J1" gate="G$1" pin="1"/>
+<pinref part="P+8" gate="1" pin="+5V"/>
+<wire x1="93.98" y1="55.88" x2="101.6" y2="55.88" width="0.1524" layer="91"/>
+</segment>
+</net>

Commit message: Add files via upload
Connections:
- net +3V3: now also U$2.V3, U$2.VCC
- net +5V: no longer U$2.VCC
Changed lines of the file:
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@@
 <part name="P+7" library="supply1" library_urn="urn:adsk.eagle:library:371" deviceset="+5V" device=""/>
 <part name="U$2" library="CH340" deviceset="CH340K" device=""/>
-<part name="P+6" library="supply1" library_urn="urn:adsk.eagle:library:371" deviceset="+5V" device=""/>
 <part name="P+8" library="supply1" library_urn="urn:adsk.eagle:library:371" deviceset="+5V" device=""/>
+<part name="+3V3" library="supply1" library_urn="urn:adsk.eagle:library:371" deviceset="+3V3" device=""/>
 </parts>
 <sheets>
@@
 <attribute name="NAME" x="43.18" y="114.3" size="1.778" layer="95"/>
 </instance>
-<instance part="P+6" gate="1" x="81.28" y="121.92" smashed="yes" rot="R270">
-<attribute name="VALUE" x="78.74" y="119.38" size="1.778" layer="96"/>
-</instance>
 <instance part="P+8" gate="1" x="104.14" y="55.88" smashed="yes" rot="R270">
 <attribute name="VALUE" x="96.52" y="55.88" size="1.778" layer="96"/>
+</instance>
+<instance part="+3V3" gate="G$1" x="81.28" y="121.92" smashed="yes" rot="R270">
+<attribute name="VALUE" x="78.74" y="119.38" size="1.778" layer="96"/>
 </instance>
 </instances>
@@
 <pinref part="U$3" gate="G$1" pin="3"/>
 <wire x1="93.98" y1="119.38" x2="88.9" y2="119.38" width="0.1524" layer="91"/>
-<label x="86.36" y="127" size="1.778" layer="95"/>
+<label x="86.36" y="119.38" size="1.778" layer="95"/>
 </segment>
 <segment>
@@
 </segment>
 <segment>
-<pinref part="U$2" gate="G$1" pin="VCC"/>
-<wire x1="66.04" y1="121.92" x2="78.74" y2="121.92" width="0.1524" layer="91"/>
-<pinref part="P+6" gate="1" pin="+5V"/>
-</segment>
-<segment>
 <pinref part="J1" gate="G$1" pin="1"/>
 <pinref part="P+8" gate="1" pin="+5V"/>
@@
 <pinref part="+3V4" gate="G$1" pin="+3V3"/>
 </segment>
-</net>
+<segment>
+<pinref part="U$2" gate="G$1" pin="VCC"/>
+<pinref part="+3V3" gate="G$1" pin="+3V3"/>
+<wire x1="66.04" y1="121.92" x2="78.74" y2="121.92" width="0.1524" layer="91"/>
+<pinref part="U$2" gate="G$1" pin="V3"/>
+<wire x1="66.04" y1="129.54" x2="78.74" y2="129.54" width="0.1524" layer="91"/>
+<wire x1="78.74" y1="129.54" x2="78.74" y2="121.92" width="0.1524" layer="91"/>
+<junction x="78.74" y="121.92"/>
+</segment>
+</net>
