File: cc2652p.brd (EAGLE design)
At the start: 25.3 x 57.3 mm, 38 parts, among them IC2 CP2102, J3 CORTEX_DEBUG_SMD, J5 TYPE-C-31-M-12, U1 MCP73831, U2 3.3V, U3 XC61CN3202MR-G

Commit message: Add files via upload
Parts:
- moved R13 3.70 mm to (3.49, 10.1), turned to 270 degrees
Routing:
- net +5V: track 56.6 -> 52.9 mm
- net GND: vias 129 -> 132

Commit message: Add files via upload
Parts:
- added R14: 10k, RC0402FR-073M6L:RESC1005X40N
- Q1: value (none) -> SI2323DS
- R1: value RC0402FR-073M6L -> 100k
- R10, R4: value RC0402FR-073M6L -> 5.1k
- R11: value RC0402FR-073M6L -> 2k
- R12, R3, R5, R9: value RC0402FR-073M6L -> 2.2k
- R13, R2: value RC0402FR-073M6L -> 10k
- R6, R7: value RC0402FR-073M6L -> 33Ohm
- R8: value RC0402FR-073M6L -> 4.7k
- U2: value 3.3V -> ap2112k-3.3
- moved R2 4.20 mm to (21.1, 17.4)
- moved U3 0.31 mm to (19.6, 15.4)
Connections:
- net N$12 renamed UVCC
- net +5V: now also R14.2
- net EN: now also R14.1
Routing:
- net EN: track 2.75 -> 7.08 mm
- net N$4: track 5.44 -> 6.86 mm
- net +5V: track 52.9 -> 53.9 mm
- net VCC: track 39.5 -> 38.5 mm
- net GND: track 27.0 -> 26.1 mm, vias 132 -> 135

Commit message: Add files via upload
Routing:
- net VCC: track 38.5 -> 48.8 mm, vias 2 -> 8
- added copper zone on layer 16, net VCC
Changed lines of the file:
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@@
 <drawing>
 <settings>
-<setting alwaysvectorfont="no"/>
+<setting alwaysvectorfont="yes"/>
 <setting verticaltext="up"/>
 </settings>
@@
 <wire x1="21.12" y1="16.918" x2="21.12" y2="15.46" width="0.2" layer="1"/>
 <wire x1="21.12" y1="15.46" x2="21.06" y2="15.4" width="0.2" layer="1"/>
+<via x="21.71" y="14.5" extent="1-16" drill="0.3"/>
+<via x="21.74" y="13.75" extent="1-16" drill="0.3"/>
+<via x="21.76" y="12.96" extent="1-16" drill="0.3"/>
+<via x="22.45" y="14.51" extent="1-16" drill="0.3"/>
+<via x="22.46" y="13.72" extent="1-16" drill="0.3"/>
+<via x="22.47" y="12.95" extent="1-16" drill="0.3"/>
+<wire x1="22.46" y1="13.72" x2="22.46" y2="14.5" width="0.3048" layer="16"/>
+<wire x1="22.45" y1="14.51" x2="22.46" y2="14.5" width="0.3048" layer="16"/>
+<wire x1="21.71" y1="14.5" x2="22.46" y2="14.5" width="0.3048" layer="16"/>
+<wire x1="22.46" y1="14.5" x2="22.49" y2="14.47" width="0.3048" layer="16"/>
+<wire x1="21.71" y1="14.5" x2="21.74" y2="14.47" width="0.3048" layer="16"/>
+<wire x1="21.74" y1="14.47" x2="21.74" y2="13.75" width="0.3048" layer="16"/>
+<wire x1="21.76" y1="13.72" x2="22.46" y2="13.72" width="0.3048" layer="16"/>
+<wire x1="21.74" y1="13.75" x2="21.76" y2="13.73" width="0.3048" layer="16"/>
+<wire x1="21.76" y1="13.73" x2="21.76" y2="13.72" width="0.3048" layer="16"/>
+<wire x1="21.76" y1="13.72" x2="21.76" y2="12.96" width="0.3048" layer="16"/>
+<wire x1="22.47" y1="12.95" x2="21.77" y2="12.95" width="0.3048" layer="16"/>
+<wire x1="21.76" y1="12.96" x2="21.77" y2="12.95" width="0.3048" layer="16"/>
+<wire x1="22.46" y1="13.72" x2="22.46" y2="12.96" width="0.3048" layer="16"/>
+<wire x1="22.47" y1="12.95" x2="22.46" y2="12.96" width="0.3048" layer="16"/>
+<polygon width="0.3048" layer="16">
+<vertex x="21.63" y="14.58"/>
+<vertex x="21.63" y="12.92"/>
+<vertex x="22.5" y="12.92"/>
+<vertex x="22.53" y="12.95"/>
+<vertex x="22.53" y="14.51"/>
+<vertex x="22.46" y="14.58"/>
+</polygon>
+<wire x1="21.63" y1="14.58" x2="21.63" y2="12.93" width="0.3048" layer="16"/>
+<wire x1="21.63" y1="12.93" x2="21.64" y2="12.92" width="0.3048" layer="16"/>
+<wire x1="21.64" y1="12.92" x2="22.42" y2="12.92" width="0.3048" layer="16"/>
+<wire x1="22.42" y1="14.48" x2="22.45" y2="14.51" width="0.3048" layer="16"/>
+<wire x1="22.42" y1="14.48" x2="22.42" y2="12.92" width="0.3048" layer="16"/>
+<wire x1="22.45" y1="14.51" x2="22.38" y2="14.58" width="0.3048" layer="16"/>
+<wire x1="22.38" y1="14.58" x2="21.63" y2="14.58" width="0.3048" layer="16"/>
 </signal>
 <signal name="EN">

Commit message: Add files via upload
Parts:
- R13: value 10k -> 100k
Connections:
- net +5V: now also J1.1
- net GND: no longer J1.1
Routing:
- net +5V: track 53.9 -> 56.8 mm
Other:
- board text added: "5V"
Changed lines of the file:
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@@
 <drawing>
 <settings>
-<setting alwaysvectorfont="yes"/>
+<setting alwaysvectorfont="no"/>
 <setting verticaltext="up"/>
 </settings>
@@
 <text x="2.9" y="14.8" size="0.8128" layer="25" font="vector" ratio="12" rot="R90">TDI</text>
 <text x="2.9" y="12" size="0.8128" layer="25" font="vector" ratio="12" rot="R90">3V3</text>
-<text x="2.9" y="9.5" size="0.8128" layer="25" font="vector" ratio="12" rot="R90">GND</text>
+<text x="2.94" y="9.86" size="0.8128" layer="25" font="vector" ratio="12" rot="R90">5V</text>
 <text x="12.9" y="0.3" size="0.8128" layer="25" font="vector" ratio="12" rot="R90">PWR</text>
 <text x="1.8" y="52.2" size="0.8128" layer="25" font="vector" ratio="12">R</text>
@@
 <attribute name="VENDOR" value="Torex Semiconductor" x="19.56" y="15.4" size="1.778" layer="27" rot="R270" display="off"/>
 </element>
-<element name="R13" library="RC0402FR-073M6L" package="RESC1005X40N" value="10k" x="3.49" y="10.11" smashed="yes" rot="R270">
+<element name="R13" library="RC0402FR-073M6L" package="RESC1005X40N" value="100k" x="3.49" y="10.11" smashed="yes" rot="R270">
 <attribute name="AVAILABILITY" value="Good" x="3.49" y="10.11" size="1.778" layer="27" rot="R270" display="off"/>
 <attribute name="DESCRIPTION" value=" RESISTOR, 0402 0.063W 1% 3M6; Resistance:3.6Mohm; Resistance Tolerance:± 1%; Power Rating:0.063W; Voltage Rating:50V; Series:RC32H; Temperature Coefficient:± 100ppm/°C; Resistor Element Type:Thick Film; Resistor Case Style:0402; No. of Pins:2; SVHC:No SVHC; Case Style:0402; External Length / Height:1mm; Temperature Coeff. +:100ppm/°C; Temperature Coeff. -:100ppm/°C; External Depth:0.35mm; External Width:0.5mm; Operating Temperature Range:-55°C to +155°C; Overload Voltage:100V " x="3.49" y="10.11" size="1.778" layer="27" rot="R270" display="off"/>
@@
 <contactref element="U$1" pad="23"/>
 <contactref element="U$1" pad="19"/>
-<contactref element="J1" pad="1"/>
 <contactref element="J1" pad="7"/>
 <contactref element="J2" pad="1"/>
@@
 <wire x1="16.97" y1="12.38" x2="17.05" y2="12.3" width="0.508" layer="1"/>
 <wire x1="16.3" y1="14" x2="16.97" y2="13.33" width="0.508" layer="1"/>
-<wire x1="3.49" y1="9.678" x2="3.54" y2="9.628" width="0.2" layer="1"/>
-<wire x1="3.54" y1="9.628" x2="3.54" y2="9.16" width="0.2" layer="1"/>
-<wire x1="3.54" y1="9.16" x2="4" y2="8.7" width="0.2" layer="1"/>
-<wire x1="4" y1="8.7" x2="4" y2="7.845" width="0.2" layer="1"/>
+<wire x1="3.54" y1="9.628" x2="3.49" y2="9.678" width="0.2" layer="1"/>
 <contactref element="R14" pad="2"/>
 <wire x1="17.25" y1="14.458" x2="16.352" y2="14.458" width="0.2" layer="1"/>
 <wire x1="16.352" y1="14.458" x2="16.3" y2="14.51" width="0.2" layer="1"/>
+<contactref element="J1" pad="1"/>
+<wire x1="3.95" y1="7.795" x2="3.95" y2="8.66" width="0.4064" layer="1"/>
+<wire x1="3.95" y1="8.66" x2="3.53" y2="9.08" width="0.4064" layer="1"/>
+<wire x1="3.53" y1="9.08" x2="3.53" y2="9.618" width="0.4064" layer="1"/>
+<wire x1="3.53" y1="9.618" x2="3.54" y2="9.628" width="0.4064" layer="1"/>
+<wire x1="3.49" y1="9.678" x2="3.458" y2="9.71" width="0.4064" layer="1"/>
+<wire x1="1.89" y1="9.71" x2="1" y2="10.6" width="0.4064" layer="1"/>
+<wire x1="3.458" y1="9.71" x2="1.89" y2="9.71" width="0.4064" layer="1"/>
 </signal>
 <signal name="UVCC">

Commit message: Add files via upload
Parts:
- added PAD1, PAD2: WIREPADSMD1,27-254, wirepad:SMD1,27-2,54
Connections:
- net GND: now also PAD1.1
- net VCC: now also PAD2.1
Routing:
- net VCC: track 48.8 -> 51.0 mm, vias 8 -> 11
- net GND: track 26.1 -> 27.3 mm, vias 135 -> 139
Other:
- board text added: "+"
- board text added: "-"
Changed lines of the file:
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@@
 <drawing>
 <settings>
-<setting alwaysvectorfont="no"/>
+<setting alwaysvectorfont="yes"/>
 <setting verticaltext="up"/>
 </settings>
-<grid distance="0.01" unitdist="mm" unit="mm" style="lines" multiple="1" display="yes" altdistance="0.1" altunitdist="mm" altunit="mm"/>
+<grid distance="0.127" unitdist="mm" unit="mm" style="lines" multiple="1" display="yes" altdistance="0.1" altunitdist="mm" altunit="mm"/>
 <layers>
 <layer number="1" name="Top" color="4" fill="1" visible="yes" active="yes"/>
+<layer number="2" name="Route2" color="1" fill="3" visible="no" active="no"/>
+<layer number="3" name="Route3" color="4" fill="3" visible="no" active="no"/>
+<layer number="4" name="Route4" color="1" fill="4" visible="no" active="no"/>
+<layer number="5" name="Route5" color="4" fill="4" visible="no" active="no"/>
+<layer number="6" name="Route6" color="1" fill="8" visible="no" active="no"/>
+<layer number="7" name="Route7" color="4" fill="8" visible="no" active="no"/>
+<layer number="8" name="Route8" color="1" fill="2" visible="no" active="no"/>
+<layer number="9" name="Route9" color="4" fill="2" visible="no" active="no"/>
+<layer number="10" name="Route10" color="1" fill="7" visible="no" active="no"/>
+<layer number="11" name="Route11" color="4" fill="7" visible="no" active="no"/>
+<layer number="12" name="Route12" color="1" fill="5" visible="no" active="no"/>
+<layer number="13" name="Route13" color="4" fill="5" visible="no" active="no"/>
+<layer number="14" name="Route14" color="1" fill="6" visible="no" active="no"/>
+<layer number="15" name="Route15" color="4" fill="6" visible="no" active="no"/>
 <layer number="16" name="Bottom" color="1" fill="1" visible="yes" active="yes"/>
 <layer number="17" name="Pads" color="2" fill="1" visible="yes" active="yes"/>
@@
 <text x="2.8" y="32.9" size="0.8128" layer="25" font="vector" ratio="12" rot="R90">13</text>
 <text x="5.4" y="26.1" size="0.8128" layer="25" font="vector" ratio="12">JTAG</text>
-<text x="3.8" y="25.5" size="1.27" layer="25" font="vector" ratio="20" rot="R90">.</text>
+<text x="3.8" y="25.5" size="1.778" layer="25" font="vector" ratio="20" rot="R90">.</text>
 <text x="21.3" y="40.3" size="1.27" layer="26" font="vector" ratio="12" rot="MR90">t.me/deaxx</text>
+<text x="17.363" y="9.693" size="1.778" layer="26" font="vector" ratio="12" rot="MR90">+</text>
+<text x="20.792" y="9.566" size="1.778" layer="26" font="vector" ratio="12" rot="MR0">-</text>
 </plain>
 <attributes>
@@
 <attribute name="PURCHASE-URL" value="https://pricing.snapeda.com/search/part/RC0402FR-073M6L/?ref=eda" x="17.25" y="14.89" size="1.778" layer="27" rot="R270" display="off"/>
 </element>
+<element name="PAD1" library="wirepad" library_urn="urn:adsk.eagle:library:412" package="SMD1,27-2,54" package3d_urn="urn:adsk.eagle:package:30839/1" value="WIREPADSMD1,27-254" x="20.34" y="8.12" smashed="yes" rot="MR0">
+<attribute name="POPULARITY" value="11" x="20.34" y="8.12" size="1.778" layer="28" rot="MR0" display="off"/>
+</element>
+<element name="PAD2" library="wirepad" library_urn="urn:adsk.eagle:library:412" package="SMD1,27-2,54" package3d_urn="urn:adsk.eagle:package:30839/1" value="WIREPADSMD1,27-254" x="18.06" y="8.13" smashed="yes" rot="MR0">
+<attribute name="POPULARITY" value="11" x="18.06" y="8.13" size="1.778" layer="28" rot="MR0" display="off"/>
+</element>
 </elements>
 <signals>
@@
 <contactref element="C1" pad="2"/>
 <contactref element="C3" pad="2"/>
-<contactref element="CN1" pad="2"/>
 <polygon width="0.15" layer="16">
 <vertex x="-0.604346875" y="51.2"/>
@@
 <via x="12.6" y="35.9" extent="1-16" drill="0.3"/>
 <via x="14.5" y="35.9" extent="1-16" drill="0.3"/>
-<wire x1="20.2" y1="7.1" x2="20.2" y2="6.3" width="0.2" layer="1"/>
 <via x="18.4" y="33.9" extent="1-16" drill="0.3"/>
-<wire x1="20.2" y1="7.1" x2="20.1" y2="7.2" width="0.2" layer="1"/>
-<wire x1="20.1" y1="7.2" x2="20.1" y2="8.1" width="0.2" layer="1"/>
 <via x="4.4" y="50.6" extent="1-16" drill="0.3"/>
 <via x="4.4" y="49" extent="1-16" drill="0.3"/>
@@
 <vertex x="-0.8" y="-0.5"/>
 </polygon>
-<wire x1="21.1001" y1="11.2" x2="22.2" y2="11.2" width="0.508" layer="1"/>
-<wire x1="22.8" y1="10.6" x2="23.9" y2="10.6" width="0.508" layer="1"/>
-<wire x1="22.2" y1="11.2" x2="22.3" y2="11.1" width="0.508" layer="1"/>
-<wire x1="22.3" y1="11.1" x2="22.8" y2="10.6" width="0.508" layer="1"/>
-<via x="22.3" y="11.1" extent="1-16" drill="0.3"/>
 <via x="11.78" y="29.94" extent="1-16" drill="0.3"/>
 <via x="3.67" y="28.67" extent="1-16" drill="0.3"/>
@@
 <via x="17.2" y="16.48" extent="1-16" drill="0.3"/>
 <via x="15.49" y="15.43" extent="1-16" drill="0.3"/>
+<contactref element="CN1" pad="2"/>
+<contactref element="PAD1" pad="1"/>
+<via x="20.193" y="9.017" extent="1-16" drill="0.3"/>
+<via x="20.193" y="8.128" extent="1-16" drill="0.3"/>
+<via x="20.193" y="7.239" extent="1-16" drill="0.3"/>
+<via x="22.291" y="11.141" extent="1-16" drill="0.3"/>
+<via x="22.291" y="10.379" extent="1-16" drill="0.3"/>
+<wire x1="21.1001" y1="11.2" x2="22.232" y2="11.2" width="0.5" layer="1"/>
+<wire x1="22.232" y1="11.2" x2="22.291" y2="11.141" width="0.4064" layer="1"/>
+<wire x1="23.9" y1="10.6" x2="23.679" y2="10.379" width="0.4064" layer="1"/>
+<wire x1="23.679" y1="10.379" x2="22.291" y2="10.379" width="0.8128" layer="1"/>
+<wire x1="22.291" y1="10.379" x2="22.232" y2="10.438" width="0.6096" layer="1"/>
+<wire x1="22.232" y1="10.438" x2="22.232" y2="11.2" width="0.6096" layer="1"/>
+<wire x1="23.9" y1="10.6" x2="23.9" y2="8.9" width="0.8128" layer="1"/>
+<wire x1="23.9" y1="8.9" x2="24.3" y2="8.5" width="0.8128" layer="1"/>
 </signal>
 <signal name="RESET">
@@
 <wire x1="20.6601" y1="15.3063" x2="20.7538" y2="15.4" width="0.2" layer="1"/>
 <wire x1="16.1" y1="8.4" x2="16.1" y2="11.2" width="0.508" layer="16"/>
-<wire x1="18.2" y1="7.1" x2="16.7" y2="7.1" width="0.6096" layer="1"/>
+<wire x1="17.907" y1="7.1" x2="16.7" y2="7.1" width="0.6096" layer="1"/>
 <wire x1="16.7" y1="7.1" x2="16.1" y2="7.7" width="0.6096" layer="1"/>
 <wire x1="16.1" y1="7.7" x2="16.1" y2="8.4" width="0.6096" layer="1"/>
@@
 <wire x1="22.45" y1="14.51" x2="22.38" y2="14.58" width="0.3048" layer="16"/>
 <wire x1="22.38" y1="14.58" x2="21.63" y2="14.58" width="0.3048" layer="16"/>
+<contactref element="PAD2" pad="1"/>
+<via x="18.22" y="9.02" extent="1-16" drill="0.3"/>
+<via x="18.22" y="8.131" extent="1-16" drill="0.3"/>
+<via x="18.22" y="7.242" extent="1-16" drill="0.3"/>
+<wire x1="18.06" y1="8.13" x2="18.219" y2="8.13" width="0.2" layer="16"/>
+<wire x1="18.219" y1="8.13" x2="18.22" y2="8.131" width="0.2" layer="16"/>
+<wire x1="18.06" y1="8.13" x2="18.22" y2="8.29" width="0.2" layer="16"/>
+<wire x1="18.22" y1="8.29" x2="18.22" y2="9.02" width="0.2" layer="16"/>
+<wire x1="18.06" y1="8.13" x2="18.22" y2="7.97" width="0.2" layer="16"/>
+<wire x1="18.22" y1="7.97" x2="18.22" y2="7.242" width="0.2" layer="16"/>
+<wire x1="18.2" y1="7.1" x2="17.907" y2="7.1" width="0.2" layer="1"/>
+<wire x1="18.2" y1="7.1" x2="18.2" y2="7.222" width="0.2" layer="1"/>
+<wire x1="18.2" y1="7.222" x2="18.22" y2="7.242" width="0.2" layer="1"/>
 </signal>
 <signal name="EN">
@@
 <wire x1="22.1" y1="3.7" x2="22.6" y2="4.2" width="0.2" layer="16"/>
 <wire x1="22.6" y1="4.2" x2="22.6" y2="8.4" width="0.2" layer="16"/>
-<wire x1="21.1001" y1="10.25" x2="22.05" y2="10.25" width="0.2" layer="1"/>
-<wire x1="22.05" y1="10.25" x2="22.6" y2="9.7" width="0.2" layer="1"/>
-<wire x1="22.6" y1="9.7" x2="22.6" y2="8.4" width="0.2" layer="1"/>
+<wire x1="21.1001" y1="10.25" x2="21.209" y2="10.1411" width="0.2" layer="1"/>
+<wire x1="21.209" y1="10.1411" x2="21.209" y2="9.652" width="0.2" layer="1"/>
+<wire x1="21.209" y1="9.652" x2="22.461" y2="8.4" width="0.2" layer="1"/>
+<wire x1="22.461" y1="8.4" x2="22.6" y2="8.4" width="0.2" layer="1"/>
 </signal>
 </signals>

Commit message: Add files via upload
Connections:
- net +3V3: now also J1.7; no longer J1.2
- net GND: now also J1.2; no longer J1.7
Routing:
- net +3V3: track 61.7 -> 47.3 mm
- net GND: vias 139 -> 137
Changed lines of the file:
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@@
 <text x="2.8" y="30.4" size="0.8128" layer="25" font="vector" ratio="12" rot="R90">14</text>
 <text x="2.9" y="27.8" size="0.8128" layer="25" font="vector" ratio="12" rot="R90">15</text>
-<text x="2.9" y="24.9" size="0.8128" layer="25" font="vector" ratio="12" rot="R90">GND</text>
+<text x="2.9" y="12.073" size="0.8128" layer="25" font="vector" ratio="12" rot="R90">GND</text>
 <text x="2.9" y="22.3" size="0.8128" layer="25" font="vector" ratio="12" rot="R90">TMS</text>
 <text x="2.9" y="19.8" size="0.8128" layer="25" font="vector" ratio="12" rot="R90">TCK</text>
 <text x="2.9" y="17.2" size="0.8128" layer="25" font="vector" ratio="12" rot="R90">TDO</text>
 <text x="2.9" y="14.8" size="0.8128" layer="25" font="vector" ratio="12" rot="R90">TDI</text>
-<text x="2.9" y="12" size="0.8128" layer="25" font="vector" ratio="12" rot="R90">3V3</text>
+<text x="2.9" y="24.827" size="0.8128" layer="25" font="vector" ratio="12" rot="R90">3V3</text>
 <text x="2.94" y="9.86" size="0.8128" layer="25" font="vector" ratio="12" rot="R90">5V</text>
 <text x="12.9" y="0.3" size="0.8128" layer="25" font="vector" ratio="12" rot="R90">PWR</text>
@@
 <text x="17.363" y="9.693" size="1.778" layer="26" font="vector" ratio="12" rot="MR90">+</text>
 <text x="20.792" y="9.566" size="1.778" layer="26" font="vector" ratio="12" rot="MR0">-</text>
+<text x="17.744" y="6.264" size="1.27" layer="26" font="vector" ratio="12" rot="MR180">BAT</text>
 </plain>
 <attributes>
@@
 <contactref element="U$1" pad="23"/>
 <contactref element="U$1" pad="19"/>
-<contactref element="J1" pad="7"/>
 <contactref element="J2" pad="1"/>
 <wire x1="3.791140625" y1="31.46016875" x2="3.791140625" y2="32.73016875" width="0.2" layer="1"/>
@@
 <via x="13.2" y="16.5" extent="1-16" drill="0.3"/>
 <via x="18.1" y="13.3" extent="1-16" drill="0.3"/>
-<via x="5" y="26.3" extent="1-16" drill="0.3"/>
 <via x="1.3" y="0.9" extent="1-16" drill="0.3"/>
 <via x="2.7" y="0.6" extent="1-16" drill="0.3"/>
@@
 </polygon>
 <via x="11.78" y="29.94" extent="1-16" drill="0.3"/>
-<via x="3.67" y="28.67" extent="1-16" drill="0.3"/>
 <wire x1="19.55" y1="20.25" x2="20.644" y2="20.25" width="0.2" layer="1"/>
 <wire x1="20.644" y1="20.25" x2="20.955" y2="19.939" width="0.2" layer="1"/>
@@
 <wire x1="23.9" y1="10.6" x2="23.9" y2="8.9" width="0.8128" layer="1"/>
 <wire x1="23.9" y1="8.9" x2="24.3" y2="8.5" width="0.8128" layer="1"/>
+<contactref element="J1" pad="2"/>
 </signal>
 <signal name="RESET">
@@
 <contactref element="R1" pad="1"/>
 <contactref element="U$1" pad="20"/>
-<contactref element="J1" pad="2"/>
 <contactref element="J3" pad="1"/>
 <wire x1="17.0999" y1="20.2001" x2="17.1" y2="20.2" width="0.4064" layer="1"/>
@@
 <wire x1="11.59675" y1="20.2" x2="17.1" y2="20.2" width="0.2" layer="16"/>
 <wire x1="10.69195" y1="19.2952" x2="11.59675" y2="20.2" width="0.2" layer="16"/>
-<via x="6.9" y="21.3" extent="1-16" drill="0.3"/>
-<wire x1="4.327" y1="24.9" x2="4.287" y2="24.94" width="0.2" layer="1"/>
+<wire x1="4.287" y1="24.94" x2="4.327" y2="24.9" width="0.2" layer="1"/>
 <wire x1="17.1" y1="29.7" x2="16.4" y2="30.4" width="0.4064" layer="16"/>
 <wire x1="16.4" y1="30.4" x2="15.6" y2="30.4" width="0.4064" layer="16"/>
@@
 <wire x1="16.2001" y1="20.25" x2="16.25" y2="20.2001" width="0.4064" layer="1"/>
 <wire x1="16.25" y1="20.2001" x2="17.0999" y2="20.2001" width="0.4064" layer="1"/>
-<wire x1="6.9" y1="21.3" x2="3.294" y2="21.3" width="0.254" layer="16"/>
-<wire x1="3.294" y1="21.3" x2="2.924" y2="20.93" width="0.254" layer="16"/>
-<wire x1="2.924" y1="20.93" x2="2.924" y2="17.9214125" width="0.254" layer="16"/>
-<wire x1="2.2192" y1="17.2166125" x2="2.2192" y2="15.1749875" width="0.254" layer="16"/>
-<wire x1="1" y1="13.9557875" x2="1" y2="13.14" width="0.254" layer="16"/>
-<wire x1="2.2192" y1="15.1749875" x2="1" y2="13.9557875" width="0.254" layer="16"/>
-<wire x1="2.924" y1="17.9214125" x2="2.2192" y2="17.2166125" width="0.254" layer="16"/>
-<wire x1="4.287" y1="24.94" x2="5.22831875" y2="24.94" width="0.254" layer="1"/>
-<wire x1="5.22831875" y1="24.94" x2="6.029825" y2="24.13849375" width="0.254" layer="1"/>
-<wire x1="6.029825" y1="24.13849375" x2="6.029825" y2="22.63361875" width="0.254" layer="1"/>
-<wire x1="6.9" y1="21.76344375" x2="6.9" y2="21.3" width="0.254" layer="1"/>
-<wire x1="6.029825" y1="22.63361875" x2="6.9" y2="21.76344375" width="0.254" layer="1"/>
-<wire x1="15.6" y1="30.4" x2="15.14" y2="30.4" width="0.254" layer="1"/>
-<wire x1="15.14" y1="30.4" x2="14.81" y2="30.73" width="0.254" layer="1"/>
-<wire x1="14.81" y1="30.73" x2="5.59669375" y2="30.73" width="0.254" layer="1"/>
-<wire x1="5.59669375" y1="30.73" x2="4.7158" y2="29.84910625" width="0.254" layer="1"/>
-<wire x1="4.287" y1="26.517" x2="4.287" y2="24.94" width="0.254" layer="1"/>
-<wire x1="4.7158" y1="29.84910625" x2="4.7158" y2="26.9458" width="0.254" layer="1"/>
-<wire x1="4.7158" y1="26.9458" x2="4.287" y2="26.517" width="0.254" layer="1"/>
+<contactref element="J1" pad="7"/>
+<wire x1="4.287" y1="24.94" x2="3.096" y2="24.94" width="0.3048" layer="1"/>
+<wire x1="3.096" y1="24.94" x2="3.048" y2="24.892" width="0.3048" layer="1"/>
+<via x="3.048" y="24.892" extent="1-16" drill="0.3"/>
+<wire x1="1" y1="25.84" x2="1.948" y2="24.892" width="0.3048" layer="16"/>
+<wire x1="1.948" y1="24.892" x2="3.048" y2="24.892" width="0.3048" layer="16"/>
+<wire x1="4.287" y1="24.94" x2="4.287" y2="27.02" width="0.3048" layer="1"/>
+<wire x1="4.287" y1="27.02" x2="4.6904" y2="27.4234" width="0.3048" layer="1"/>
+<wire x1="4.6904" y1="29.859625" x2="5.540375" y2="30.7096" width="0.3048" layer="1"/>
+<wire x1="5.540375" y1="30.7096" x2="15.2904" y2="30.7096" width="0.3048" layer="1"/>
+<wire x1="15.2904" y1="30.7096" x2="15.5476" y2="30.4524" width="0.3048" layer="1"/>
+<wire x1="4.6904" y1="27.4234" x2="4.6904" y2="29.859625" width="0.3048" layer="1"/>
 </signal>
 <signal name="CC2">

Commit message: Add files via upload
Parts:
- moved R1 2.62 mm to (11.6, 20.1)
- moved C3 1.66 mm to (13.1, 19.4)
Connections:
- net RESET: now also J3.10
Routing:
- net VCC: track 51.0 -> 73.1 mm
- net +3V3: track 47.3 -> 43.6 mm
- net GND: track 27.3 -> 25.1 mm, vias 137 -> 136
- net RESET: track 39.6 -> 40.2 mm
Other:
- board text added: "+5V"
- board text added: "DIO10"
- board text added: "DIO11"
- board text added: "DIO12"
- board text added: "DIO13"
- board text added: "DIO14"
- board text added: "DIO15"
- board text added: "DIO18"
- board text added: "DIO19"
- board text added: "DIO20"
- board text added: "DIO21"
- board text added: "DIO22"
- board text added: "DIO23"
- board text added: "DIO24"
- board text added: "DIO25"
- board text added: "DIO26"
- board text added: "DIO27"
- board text added: "DIO28"
- board text added: "DIO29"
- board text added: "DIO30"
- board text added: "DIO7"
- board text added: "DIO8"
- board text added: "DIO9"
- board text added: "RESET"

Commit message: Add files via upload
Parts:
- removed C3: 0.1uF, SparkFun-Capacitors:0603
- removed R1: 100k, RC0402FR-073M6L:RESC1005X40N
Connections:
- removed net N$4: C4.1, IC2.6, R9.1
- net +3V3: now also C4.1, IC2.6, IC2.7, R9.1; no longer R1.1
- net +5V: no longer IC2.7
- net GND: no longer C3.2
- net RESET: no longer C3.1, R1.2
Routing:
- net +3V3: track 43.6 -> 56.3 mm
- net N$4: track 6.86 -> 0.00 mm
- net +5V: track 56.8 -> 53.5 mm, vias 4 -> 3
- net GND: vias 136 -> 139
