File: cc2652p.brd (EAGLE design)
At the start: 25.3 x 57.3 mm, 39 parts, among them IC2 CP2102, J3 CORTEX_DEBUG_SMD, J5 TYPE-C-31-M-12, Q1 SI2323DS, U1 MCP73831, U2 ap2112k-3.3, U3 XC61CN3202MR-G

Commit message: Add files via upload
Parts:
- added C3: 100n, discretes-dev:CAPC1005X40N
- added R1: 2.2k, RC0402FR-073M6L:RESC1005X40N
- added R15, R16: 0, RC0402FR-073M6L:RESC1005X40N
- added U$2: MX25R8035FM1IL0, W25Q80BVSNIG:SO-8
Connections:
- new net N$12: R15.2, U$2.7
- new net N$15: R16.1, U$2.3
- new net N$17: R1.2, U$2.1
- net +3V3: now also C3.2, R1.1, R15.1, R16.2, U$2.8
- net DIO_10: now also U$2.6
- net DIO_8: now also U$2.2
- net DIO_9: now also U$2.5
- net GND: now also C3.1, U$2.4
Routing:
- net +3V3: track 56.3 -> 83.5 mm
- net DIO_8: track 18.0 -> 33.1 mm, vias 2 -> 3
- net N$15: track 0.00 -> 10.00 mm
- net DIO_9: track 3.97 -> 13.2 mm, vias 0 -> 1
- net DIO_10: track 3.09 -> 10.2 mm, vias 0 -> 1
- net N$12: track 0.00 -> 6.67 mm
- net DIO_14: track 37.8 -> 34.4 mm
- net N$17: track 0.00 -> 1.41 mm
- net GND: vias 139 -> 103

Commit message: Add files via upload
Connections:
- removed net N$17: R1.2, U$2.1
- net DIO_20: now also R1.2, U$2.1
Routing:
- net DIO_20: track 13.2 -> 35.7 mm, vias 0 -> 1
- net N$17: track 1.41 -> 0.00 mm
- net GND: vias 103 -> 97
Changed lines of the file:
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@@
 <contactref element="C3" pad="1"/>
 <contactref element="U$2" pad="4"/>
-<via x="16.41" y="39.4" extent="1-16" drill="0.3"/>
-<via x="16.41" y="37.5" extent="1-16" drill="0.3"/>
-<via x="16.41" y="35.9" extent="1-16" drill="0.3"/>
 <via x="8.74" y="50.6" extent="1-16" drill="0.3"/>
 <via x="11.28" y="50.6" extent="1-16" drill="0.3"/>
@@
 <via x="14.505" y="37.495" extent="1-16" drill="0.3"/>
 <via x="14.505" y="35.9" extent="1-16" drill="0.3"/>
-<via x="16.495" y="41.1" extent="1-16" drill="0.3"/>
-<via x="14.59" y="41.1" extent="1-16" drill="0.3"/>
 <via x="10.902" y="43.845" extent="1-16" drill="0.3"/>
-<via x="13.315" y="43.845" extent="1-16" drill="0.3"/>
-<via x="13.315" y="46.004" extent="1-16" drill="0.3"/>
 <via x="4.422" y="47.171" extent="1-16" drill="0.3"/>
 <via x="18.4" y="42.878" extent="1-16" drill="0.3"/>
+<via x="16.114" y="41.1" extent="1-16" drill="0.3"/>
 </signal>
 <signal name="RESET">
@@
 <via x="19.2" y="23.6" extent="1-16" drill="0.3"/>
 <via x="17.1" y="34" extent="1-16" drill="0.3"/>
-<wire x1="17.5556" y1="25.2444" x2="17.5556" y2="29.88871875" width="0.2" layer="16"/>
-<wire x1="17.5556" y1="29.88871875" x2="16.5524" y2="30.89191875" width="0.2" layer="16"/>
+<wire x1="17.5556" y1="25.2444" x2="17.5556" y2="30.39671875" width="0.2" layer="16"/>
+<wire x1="17.5556" y1="30.39671875" x2="16.5524" y2="31.39991875" width="0.2" layer="16"/>
 <wire x1="16.5524" y1="33.4524" x2="17.1" y2="34" width="0.2" layer="16"/>
 <wire x1="19.2" y1="23.6" x2="17.5556" y2="25.2444" width="0.2" layer="16"/>
-<wire x1="16.5524" y1="30.89191875" x2="16.5524" y2="33.4524" width="0.2" layer="16"/>
+<wire x1="16.5524" y1="31.39991875" x2="16.5524" y2="33.4524" width="0.2" layer="16"/>
 </signal>
 <signal name="TMS">
@@
 <wire x1="21.59721875" y1="27.2" x2="22.3554" y2="26.44181875" width="0.2" layer="1"/>
 <wire x1="22.3554" y1="26.44181875" x2="22.3554" y2="25.20019375" width="0.2" layer="1"/>
+<contactref element="U$2" pad="1"/>
+<contactref element="R1" pad="2"/>
+<wire x1="15.799" y1="47.371" x2="15.799" y2="45.9992" width="0.2" layer="16"/>
+<wire x1="15.799" y1="45.9992" x2="15.8242" y2="45.974" width="0.2" layer="16"/>
+<wire x1="15.8242" y1="45.974" x2="13.843" y2="45.974" width="0.2" layer="16"/>
+<wire x1="13.843" y1="45.974" x2="13.335" y2="45.466" width="0.2" layer="16"/>
+<wire x1="13.335" y1="45.466" x2="13.335" y2="41.41131875" width="0.2" layer="16"/>
+<wire x1="16.891" y1="30.05494375" x2="16.891" y2="29.972" width="0.2" layer="16"/>
+<wire x1="16.2" y1="30.74594375" x2="16.891" y2="30.05494375" width="0.2" layer="16"/>
+<wire x1="16.2" y1="38.54631875" x2="16.2" y2="30.74594375" width="0.2" layer="16"/>
+<wire x1="13.335" y1="41.41131875" x2="16.2" y2="38.54631875" width="0.2" layer="16"/>
+<via x="16.891" y="29.972" extent="1-16" drill="0.3"/>
+<wire x1="16.8907375" y1="28.57803125" x2="16.8907375" y2="29.9717375" width="0.2" layer="1"/>
+<wire x1="16.8907375" y1="29.9717375" x2="16.891" y2="29.972" width="0.2" layer="1"/>
 </signal>
 <signal name="DIO_21">
@@
 <wire x1="17.907" y1="48.641" x2="15.799" y2="48.641" width="0.2" layer="16"/>
 </signal>
-<signal name="N$17">
-<contactref element="U$2" pad="1"/>
-<contactref element="R1" pad="2"/>
-<wire x1="15.799" y1="47.371" x2="15.799" y2="45.9992" width="0.2" layer="16"/>
-<wire x1="15.799" y1="45.9992" x2="15.8242" y2="45.974" width="0.2" layer="16"/>
-</signal>
 </signals>

Commit message: Add files via upload
Parts:
- added C13: 220uF, Capacitor:CAPM7343X310
Connections:
- net +3V3: now also C13.1
- net GND: now also C13.2, J3.9; no longer J3.3, J3.5
Routing:
- net DIO_20: track 35.7 -> 38.7 mm
- net GND: vias 97 -> 96
Other:
- outline, holes or cut-outs redrawn
- board text added: "DIO12/RX"
- board text added: "DIO13/TX"
- board text added: "DIO16/TDO"
- board text added: "DIO17/TDI"
- board text removed: "DIO12"
- board text removed: "DIO13"

Commit message: Add files via upload
Parts:
- added PSM: (no value), jumper:SJ
Connections:
- new net V+: C2.1, C4.1, IC2.6, IC2.7, PSM.1, R9.1, U2.5
- net +3V3: now also PSM.2; no longer C2.1, C4.1, IC2.6, IC2.7, R9.1, U2.5
Routing:
- net V+: track 0.00 -> 23.7 mm, vias 0 -> 2
- net +3V3: track 83.7 -> 63.4 mm, vias 4 -> 2
Other:
- board text added: "PSM"

Commit message: Add files via upload
Parts:
- removed PSM: (no value), jumper:SJ
- added Q2: SI2323DS, SI2323DS:SOT23
Connections:
- net +3V3: now also Q2.2; no longer PSM.2
- net GND: now also Q2.1
- net V+: now also Q2.3; no longer PSM.1
Routing:
- net +3V3: track 63.4 -> 66.7 mm, vias 2 -> 3
- net V+: track 23.7 -> 25.1 mm
- net GND: vias 96 -> 100
Other:
- board text removed: "PSM"

Commit message: Add files via upload
Parts:
- removed Q2: SI2323DS, SI2323DS:SOT23
- added PSM: PSM, pimoroni-misc:SOLDER_JUMPER_CLOSED
Connections:
- net +3V3: now also PSM.2; no longer Q2.2
- net GND: no longer Q2.1
- net V+: now also PSM.1; no longer Q2.3
Routing:
- net +3V3: track 66.7 -> 61.1 mm, vias 3 -> 2
- net V+: track 25.1 -> 22.7 mm
- net GND: vias 100 -> 98
Other:
- board text added: "PSM"
Changed lines of the file:
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@@
 <hole x="1.778" y="55.245" drill="2.6"/>
 <hole x="23.114" y="55.245" drill="2.6"/>
+<text x="15.053" y="20.322" size="1.016" layer="26" font="vector" ratio="12" rot="MR0">PSM</text>
 </plain>
 <attributes>
@@
 <attribute name="VOLTAGE_RATING" value="" x="21.209" y="48.514" size="1.778" layer="28" rot="MR0" display="off"/>
 </element>
-<element name="Q2" library="SI2323DS" package="SOT23" value="SI2323DS" x="11.557" y="18.796" smashed="yes">
-<attribute name="AVAILABILITY" value="Unavailable" x="11.557" y="18.796" size="1.778" layer="27" display="off"/>
-<attribute name="DESCRIPTION" value=" P-Channel 20V 3.7A (Ta) 750mW (Ta) Surface Mount SOT-23-3 (TO-236) " x="11.557" y="18.796" size="1.778" layer="27" display="off"/>
-<attribute name="MF" value="Vishay Siliconix" x="11.557" y="18.796" size="1.778" layer="27" display="off"/>
-<attribute name="MP" value="SI2323DS" x="11.557" y="18.796" size="1.778" layer="27" display="off"/>
-<attribute name="NAME" x="12.32043125" y="19.94043125" size="0.8128" layer="25" ratio="18"/>
-<attribute name="PACKAGE" value="SOT-23-3 Vishay Siliconix" x="11.557" y="18.796" size="1.778" layer="27" display="off"/>
-<attribute name="PRICE" value="None" x="11.557" y="18.796" size="1.778" layer="27" display="off"/>
-</element>
+<element name="PSM" library="pimoroni-misc" package="SOLDER_JUMPER_CLOSED" value="PSM" x="16.002" y="19.685" smashed="yes" rot="MR138"/>
 </elements>
 <signals>
@@
 <via x="10.764" y="27.273" extent="1-16" drill="0.3"/>
 <contactref element="C13" pad="2"/>
-<contactref element="Q2" pad="1"/>
-<via x="8.921" y="18.93" extent="1-16" drill="0.3"/>
-<via x="8.921" y="17.533" extent="1-16" drill="0.3"/>
 <via x="7.778" y="17.533" extent="1-16" drill="0.3"/>
-<via x="12.731" y="16.39" extent="1-16" drill="0.3"/>
 <via x="19.462" y="17.279" extent="1-16" drill="0.3"/>
 <via x="20.986" y="18.93" extent="1-16" drill="0.3"/>
 <via x="14.382" y="22.232" extent="1-16" drill="0.3"/>
-<via x="13.62" y="18.041" extent="1-16" drill="0.3"/>
+<via x="12.35" y="19.819" extent="1-16" drill="0.3"/>
+<via x="12.35" y="17.533" extent="1-16" drill="0.3"/>
 </signal>
 <signal name="RESET">
@@
 <wire x1="15.6" y1="30.4" x2="15.6" y2="38.9562" width="0.4064" layer="16"/>
 <wire x1="15.6" y1="38.9562" x2="15.5672" y2="38.989" width="0.4064" layer="16"/>
-<contactref element="Q2" pad="2"/>
-<wire x1="12.507" y1="17.696" x2="12.507" y2="18.603" width="0.4064" layer="1"/>
-<wire x1="12.954" y1="19.05" x2="12.507" y2="18.603" width="0.4064" layer="1"/>
-<wire x1="12.954" y1="19.05" x2="13.081" y2="19.05" width="0.4064" layer="1"/>
-<via x="13.081" y="19.05" extent="1-16" drill="0.3"/>
-<wire x1="17.1" y1="20.656" x2="15.494" y2="19.05" width="0.4064" layer="16"/>
-<wire x1="15.494" y1="19.05" x2="13.081" y2="19.05" width="0.4064" layer="16"/>
 <wire x1="17.1" y1="27.35" x2="17.1" y2="20.656" width="0.4064" layer="16"/>
+<contactref element="PSM" pad="2"/>
+<wire x1="17.1" y1="20.656" x2="16.634590625" y2="20.190590625" width="0.4064" layer="16"/>
+<wire x1="16.559403125" y1="20.190590625" x2="16.522203125" y2="20.153390625" width="0.4064" layer="16"/>
+<wire x1="16.634590625" y1="20.190590625" x2="16.559403125" y2="20.190590625" width="0.4064" layer="16"/>
 </signal>
 <signal name="CC2">
@@
 <wire x1="11.2" y1="11.8" x2="11.7" y2="11.8" width="0.3048" layer="1"/>
 <wire x1="11.7" y1="11.8" x2="11.7" y2="11.16" width="0.3048" layer="1"/>
-<contactref element="Q2" pad="3"/>
-<wire x1="14.65" y1="20.25" x2="13.138" y2="20.25" width="0.4064" layer="1"/>
-<wire x1="12.784" y1="19.896" x2="11.557" y2="19.896" width="0.4064" layer="1"/>
-<wire x1="13.138" y1="20.25" x2="12.784" y2="19.896" width="0.4064" layer="1"/>
-<wire x1="11.557" y1="19.896" x2="11.473" y2="19.812" width="0.4064" layer="1"/>
-<wire x1="11.473" y1="19.812" x2="10.668" y2="19.812" width="0.4064" layer="1"/>
-<wire x1="10.668" y1="19.812" x2="10.033" y2="19.177" width="0.4064" layer="1"/>
-<wire x1="10.033" y1="19.177" x2="10.033" y2="18.923" width="0.4064" layer="1"/>
-<via x="10.033" y="18.923" extent="1-16" drill="0.3"/>
-<wire x1="10.033" y1="18.923" x2="11.557" y2="18.923" width="0.4064" layer="16"/>
-<wire x1="13.462" y1="17.018" x2="13.462" y2="11.684" width="0.4064" layer="16"/>
-<wire x1="13.462" y1="11.684" x2="12.573" y2="10.795" width="0.4064" layer="16"/>
+<wire x1="12.573" y1="10.795" x2="13.462" y2="11.684" width="0.4064" layer="16"/>
 <wire x1="12.573" y1="10.795" x2="12.446" y2="10.795" width="0.4064" layer="16"/>
-<wire x1="11.557" y1="18.923" x2="13.462" y2="17.018" width="0.4064" layer="16"/>
+<contactref element="PSM" pad="1"/>
+<wire x1="15.4818" y1="19.21660625" x2="15.4818" y2="19.0378" width="0.4064" layer="16"/>
+<wire x1="13.462" y1="17.19680625" x2="15.44048125" y2="19.1752875" width="0.4064" layer="16"/>
+<wire x1="15.44048125" y1="19.1752875" x2="15.44048125" y2="19.179403125" width="0.4064" layer="16"/>
+<wire x1="15.44048125" y1="19.179403125" x2="15.477684375" y2="19.21660625" width="0.4064" layer="16"/>
+<wire x1="15.477684375" y1="19.21660625" x2="15.4818" y2="19.21660625" width="0.4064" layer="16"/>
+<wire x1="13.462" y1="11.684" x2="13.462" y2="17.19680625" width="0.4064" layer="16"/>
+<wire x1="15.4818" y1="19.21660625" x2="14.37840625" y2="20.32" width="0.4064" layer="16"/>
+<wire x1="14.37840625" y1="20.32" x2="13.335" y2="20.32" width="0.4064" layer="16"/>
+<via x="13.335" y="20.32" extent="1-16" drill="0.3"/>
+<wire x1="13.335" y1="20.32" x2="14.58" y2="20.32" width="0.4064" layer="1"/>
+<wire x1="14.58" y1="20.32" x2="14.65" y2="20.25" width="0.4064" layer="1"/>
 </signal>
 </signals>

Commit message: Add files via upload
Parts:
- removed PSM: PSM, pimoroni-misc:SOLDER_JUMPER_CLOSED
- added Q2: SI2323DS, SI2323DS:SOT23
- added R17, R18: 100k, RC0402FR-073M6L:RESC1005X40N
- added SJ1: PSM, pimoroni-misc:SMALL_SOLDER_JUMPER_CLOSED
- added U4: MMDT2907A-7-F, MMDT2907A-7-F:SOT65P210X110-6N
Connections:
- new net N$10: Q2.1, R17.2, U4.6
- new net N$4: R18.2, U4.2, U4.3, U4.5
- net +3V3: now also Q2.2, SJ1.2, U4.1; no longer PSM.2
- net GND: now also R17.1, R18.1
- net V+: now also Q2.3, SJ1.1, U4.4; no longer PSM.1
Routing:
- net N$10: track 0.00 -> 10.4 mm, vias 0 -> 1
- net +3V3: track 61.1 -> 68.9 mm
- net N$4: track 0.00 -> 5.11 mm, vias 0 -> 1
- net V+: track 22.7 -> 27.8 mm, vias 2 -> 3
- net GND: vias 98 -> 96
Other:
- board text removed: "PSM"

Commit message: Add files via upload
Parts:
- added U5: MX25R8035FZUIL0, MX25R8035FZUIL0:PSON50P200X300X60-9N
- D5: value (none) -> MBR0540
- moved D2 1.54 mm to (22.7, 49.9)
- moved C3 1.54 mm to (9.15, 45.9)
- moved R1 1.54 mm to (15.0, 45.9)
- moved R12 1.54 mm to (13.5, 5.40)
- moved R16 1.54 mm to (15.0, 47.1)
- moved R7 1.54 mm to (8.03, 8.30)
- moved R9 1.54 mm to (11.9, 5.40)
- moved RST 1.54 mm to (12.0, 22.2)
- moved BTN1 1.54 mm to (19.6, 22.1)
- moved BTN2 1.54 mm to (15.8, 22.1)
- moved C13 1.54 mm to (12.1, 37.5)
- moved D1 1.54 mm to (1.63, 49.9)
- moved D4 1.54 mm to (4.43, 12.0)
- moved D5 1.54 mm to (14.7, 13.8)
- moved PAD2 1.54 mm to (17.7, 6.63)
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Connections:
- net +3V3: now also U5.8
- net DIO_10: now also U5.6
- net DIO_20: now also U5.1
- net DIO_8: now also U5.2
- net DIO_9: now also U5.5
- net GND: now also J5.S5, J5.S6, U5.4, U5.9; no longer J5.S1, J5.S2
- net N$12: now also U5.7
- net N$15: now also U5.3
Routing:
- net DIO_10: track 10.2 -> 12.8 mm
- net N$15: track 10.00 -> 12.3 mm
- net DIO_8: track 33.1 -> 35.4 mm
- net N$12: track 6.67 -> 8.98 mm
- net +3V3: track 68.9 -> 71.0 mm
- net GND: track 25.1 -> 26.9 mm
- net DIO_9: track 13.2 -> 14.1 mm
