File: cc2652p.sch (EAGLE design)
At the start: 38 parts, among them IC2 CP2102, J3 CORTEX_DEBUG_SMD, J5 TYPE-C-31-M-12, U1 MCP73831, U2 3.3V, U3 XC61CN3202MR-G

Commit message: Add files via upload
Parts:
- added R14: 10k, RC0402FR-073M6L:RC0402FR-073M6L
- Q1: value (none) -> SI2323DS
- R1: value RC0402FR-073M6L -> 100k
- R10, R4: value RC0402FR-073M6L -> 5.1k
- R11: value RC0402FR-073M6L -> 2k
- R12, R3, R5, R9: value RC0402FR-073M6L -> 2.2k
- R13, R2: value RC0402FR-073M6L -> 10k
- R6, R7: value RC0402FR-073M6L -> 33Ohm
- R8: value RC0402FR-073M6L -> 4.7k
- U2: value 3.3V -> ap2112k-3.3
Connections:
- net N$12 renamed UVCC
- net +5V: now also R14.2
- net EN: now also R14.1
Other:
- moved on the sheet: BTN1, BTN2, C1, C2, C3, C4, CN1, D1, D2, D3, D4, D5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

Commit message: Add files via upload
Parts:
- R13: value 10k -> 100k
Connections:
- net +5V: now also J1.1
- net GND: no longer J1.1
Changed lines of the file:
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@@
 <part name="U3" library="XC61CN3202MRG" deviceset="XC61CN3202MR-G" device=""/>
 <part name="GND23" library="supply1" library_urn="urn:adsk.eagle:library:371" deviceset="GND" device=""/>
-<part name="R13" library="RC0402FR-073M6L" deviceset="RC0402FR-073M6L" device="" value="10k"/>
+<part name="R13" library="RC0402FR-073M6L" deviceset="RC0402FR-073M6L" device="" value="100k"/>
 <part name="GND25" library="supply1" library_urn="urn:adsk.eagle:library:371" deviceset="GND" device=""/>
 <part name="R14" library="RC0402FR-073M6L" deviceset="RC0402FR-073M6L" device="" value="10k"/>
 <part name="P+7" library="supply1" library_urn="urn:adsk.eagle:library:371" deviceset="+5V" device=""/>
+<part name="P+8" library="supply1" library_urn="urn:adsk.eagle:library:371" deviceset="+5V" device=""/>
 </parts>
 <sheets>
@@
 <instance part="P+7" gate="1" x="96.52" y="198.12" smashed="yes">
 <attribute name="VALUE" x="93.98" y="193.04" size="1.778" layer="96" rot="R90"/>
+</instance>
+<instance part="P+8" gate="1" x="104.14" y="55.88" smashed="yes" rot="R270">
+<attribute name="VALUE" x="96.52" y="55.88" size="1.778" layer="96"/>
 </instance>
 </instances>
@@
 </segment>
 <segment>
-<pinref part="J1" gate="G$1" pin="1"/>
-<wire x1="93.98" y1="55.88" x2="101.6" y2="55.88" width="0.1524" layer="91"/>
-<label x="96.52" y="55.88" size="1.778" layer="95"/>
-</segment>
-<segment>
 <pinref part="J1" gate="G$1" pin="7"/>
 <wire x1="93.98" y1="71.12" x2="101.6" y2="71.12" width="0.1524" layer="91"/>
@@
 <wire x1="96.52" y1="193.04" x2="96.52" y2="195.58" width="0.1524" layer="91"/>
 </segment>
-</net>
+<segment>
+<pinref part="J1" gate="G$1" pin="1"/>
+<wire x1="93.98" y1="55.88" x2="101.6" y2="55.88" width="0.1524" layer="91"/>
+<pinref part="P+8" gate="1" pin="+5V"/>
+</segment>
+</net>

Commit message: Add files via upload
Parts:
- added PAD1, PAD2: WIREPADSMD1,27-254, wirepad:WIREPADSMD1,27-254
Connections:
- net GND: now also PAD1.P
- net VCC: now also PAD2.P
Other:
- moved on the sheet: CN1
Changed lines of the file:
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@@
 <layers>
 <layer number="1" name="Top" color="4" fill="1" visible="no" active="no"/>
+<layer number="2" name="Route2" color="1" fill="3" visible="no" active="no"/>
+<layer number="3" name="Route3" color="4" fill="3" visible="no" active="no"/>
+<layer number="4" name="Route4" color="1" fill="4" visible="no" active="no"/>
+<layer number="5" name="Route5" color="4" fill="4" visible="no" active="no"/>
+<layer number="6" name="Route6" color="1" fill="8" visible="no" active="no"/>
+<layer number="7" name="Route7" color="4" fill="8" visible="no" active="no"/>
+<layer number="8" name="Route8" color="1" fill="2" visible="no" active="no"/>
+<layer number="9" name="Route9" color="4" fill="2" visible="no" active="no"/>
+<layer number="10" name="Route10" color="1" fill="7" visible="no" active="no"/>
+<layer number="11" name="Route11" color="4" fill="7" visible="no" active="no"/>
+<layer number="12" name="Route12" color="1" fill="5" visible="no" active="no"/>
+<layer number="13" name="Route13" color="4" fill="5" visible="no" active="no"/>
+<layer number="14" name="Route14" color="1" fill="6" visible="no" active="no"/>
+<layer number="15" name="Route15" color="4" fill="6" visible="no" active="no"/>
 <layer number="16" name="Bottom" color="1" fill="1" visible="no" active="no"/>
 <layer number="17" name="Pads" color="2" fill="1" visible="no" active="no"/>
@@
 <part name="P+7" library="supply1" library_urn="urn:adsk.eagle:library:371" deviceset="+5V" device=""/>
 <part name="P+8" library="supply1" library_urn="urn:adsk.eagle:library:371" deviceset="+5V" device=""/>
+<part name="PAD1" library="wirepad" library_urn="urn:adsk.eagle:library:412" deviceset="WIREPAD" device="SMD1,27-254" package3d_urn="urn:adsk.eagle:package:30839/1"/>
+<part name="PAD2" library="wirepad" library_urn="urn:adsk.eagle:library:412" deviceset="WIREPAD" device="SMD1,27-254" package3d_urn="urn:adsk.eagle:package:30839/1"/>
 </parts>
 <sheets>
@@
 <attribute name="VALUE" x="142.24" y="185.166" size="1.778" layer="96" font="vector" align="top-left"/>
 </instance>
-<instance part="CN1" gate="G$1" x="246.38" y="200.66" smashed="yes">
-<attribute name="NAME" x="240.03" y="206.375" size="1.778" layer="95"/>
-<attribute name="VALUE" x="240.03" y="195.58" size="1.778" layer="96"/>
-</instance>
-<instance part="GND5" gate="1" x="231.14" y="210.82" smashed="yes" rot="R180">
-<attribute name="VALUE" x="233.68" y="213.36" size="1.778" layer="96" rot="R180"/>
+<instance part="CN1" gate="G$1" x="246.38" y="198.12" smashed="yes">
+<attribute name="NAME" x="240.03" y="203.835" size="1.778" layer="95"/>
+<attribute name="VALUE" x="240.03" y="193.04" size="1.778" layer="96"/>
+</instance>
+<instance part="GND5" gate="1" x="233.68" y="208.28" smashed="yes" rot="R180">
+<attribute name="VALUE" x="236.22" y="210.82" size="1.778" layer="96" rot="R180"/>
 </instance>
 <instance part="BTN1" gate="G$1" x="111.76" y="27.94" smashed="yes">
@@
 <instance part="P+8" gate="1" x="104.14" y="55.88" smashed="yes" rot="R270">
 <attribute name="VALUE" x="96.52" y="55.88" size="1.778" layer="96"/>
+</instance>
+<instance part="PAD1" gate="G$1" x="226.06" y="205.74" smashed="yes" rot="R270">
+<attribute name="NAME" x="227.9142" y="206.883" size="1.778" layer="95" rot="R270"/>
+</instance>
+<instance part="PAD2" gate="G$1" x="233.68" y="195.58" smashed="yes" rot="R90">
+<attribute name="NAME" x="231.8258" y="194.437" size="1.778" layer="95" rot="R90"/>
 </instance>
 </instances>
@@
 <pinref part="U1" gate="G$1" pin="VBAT"/>
 <wire x1="215.9" y1="198.12" x2="233.68" y2="198.12" width="0.1524" layer="91"/>
-<wire x1="233.68" y1="198.12" x2="233.68" y2="200.66" width="0.1524" layer="91"/>
 <pinref part="CN1" gate="G$1" pin="2"/>
-<wire x1="233.68" y1="200.66" x2="243.84" y2="200.66" width="0.1524" layer="91"/>
+<wire x1="233.68" y1="198.12" x2="243.84" y2="198.12" width="0.1524" layer="91"/>
 <label x="215.9" y="198.12" size="1.778" layer="95"/>
+<pinref part="PAD2" gate="G$1" pin="P"/>
+<junction x="233.68" y="198.12"/>
 </segment>
 <segment>
@@
 <wire x1="86.36" y1="25.4" x2="86.36" y2="22.86" width="0.1524" layer="91"/>
 <pinref part="GND8" gate="1" pin="GND"/>
-</segment>
-<segment>
-<pinref part="CN1" gate="G$1" pin="1"/>
-<wire x1="243.84" y1="203.2" x2="231.14" y2="203.2" width="0.1524" layer="91"/>
-<wire x1="231.14" y1="203.2" x2="231.14" y2="208.28" width="0.1524" layer="91"/>
-<pinref part="GND5" gate="1" pin="GND"/>
 </segment>
 <segment>
@@
 <pinref part="GND25" gate="1" pin="GND"/>
 </segment>
+<segment>
+<pinref part="CN1" gate="G$1" pin="1"/>
+<wire x1="243.84" y1="200.66" x2="233.68" y2="200.66" width="0.1524" layer="91"/>
+<pinref part="PAD1" gate="G$1" pin="P"/>
+<wire x1="233.68" y1="200.66" x2="226.06" y2="200.66" width="0.1524" layer="91"/>
+<wire x1="226.06" y1="200.66" x2="226.06" y2="203.2" width="0.1524" layer="91"/>
+<pinref part="GND5" gate="1" pin="GND"/>
+<wire x1="233.68" y1="205.74" x2="233.68" y2="200.66" width="0.1524" layer="91"/>
+<junction x="233.68" y="200.66"/>
+</segment>
 </net>

Commit message: Add files via upload
Connections:
- net +3V3: now also J1.7; no longer J1.2
- net GND: now also J1.2; no longer J1.7
Changed lines of the file:
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@@
 <attribute name="VALUE" x="182.88" y="195.58" size="1.778" layer="96" rot="R180"/>
 </instance>
-<instance part="+3V2" gate="G$1" x="104.14" y="58.42" smashed="yes" rot="R270">
-<attribute name="VALUE" x="96.52" y="58.42" size="1.778" layer="96"/>
+<instance part="+3V2" gate="G$1" x="104.14" y="71.12" smashed="yes" rot="R270">
+<attribute name="VALUE" x="96.52" y="71.12" size="1.778" layer="96"/>
 </instance>
 <instance part="R12" gate="G$1" x="185.42" y="180.34" smashed="yes" rot="R90">
@@
 </segment>
 <segment>
-<pinref part="J1" gate="G$1" pin="7"/>
-<wire x1="93.98" y1="71.12" x2="101.6" y2="71.12" width="0.1524" layer="91"/>
-<label x="96.52" y="71.12" size="1.778" layer="95"/>
-</segment>
-<segment>
 <pinref part="J2" gate="G$1" pin="1"/>
 <wire x1="116.84" y1="55.88" x2="124.46" y2="55.88" width="0.1524" layer="91"/>
@@
 <wire x1="233.68" y1="205.74" x2="233.68" y2="200.66" width="0.1524" layer="91"/>
 <junction x="233.68" y="200.66"/>
+</segment>
+<segment>
+<pinref part="J1" gate="G$1" pin="2"/>
+<wire x1="93.98" y1="58.42" x2="101.6" y2="58.42" width="0.1524" layer="91"/>
+<label x="96.52" y="58.42" size="1.778" layer="95"/>
 </segment>
 </net>
@@
 </segment>
 <segment>
-<pinref part="J1" gate="G$1" pin="2"/>
-<wire x1="93.98" y1="58.42" x2="101.6" y2="58.42" width="0.1524" layer="91"/>
-<pinref part="+3V2" gate="G$1" pin="+3V3"/>
-</segment>
-<segment>
 <pinref part="J3" gate="G$1" pin="VCC"/>
 <wire x1="149.86" y1="63.5" x2="142.24" y2="63.5" width="0.1524" layer="91"/>
@@
 <pinref part="+3V4" gate="G$1" pin="+3V3"/>
 </segment>
-</net>
+<segment>
+<pinref part="J1" gate="G$1" pin="7"/>
+<wire x1="93.98" y1="71.12" x2="101.6" y2="71.12" width="0.1524" layer="91"/>
+<pinref part="+3V2" gate="G$1" pin="+3V3"/>
+</segment>
+</net>

Commit message: Add files via upload
Connections:
- net RESET: now also J3.!RESET
Changed lines of the file:
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@@
 <label x="116.84" y="71.12" size="1.778" layer="95"/>
+</segment>
+<segment>
+<pinref part="J3" gate="G$1" pin="!RESET"/>
+<wire x1="182.88" y1="53.34" x2="190.5" y2="53.34" width="0.1524" layer="91"/>
+<label x="185.42" y="53.34" size="1.778" layer="95"/>
 </segment>
 </net>

Commit message: Add files via upload
Parts:
- removed C3: 0.1uF, SparkFun-Capacitors:0.1UF-0603-25V-(+80/-20%)
- removed R1: 100k, RC0402FR-073M6L:RC0402FR-073M6L
Connections:
- removed net N$4: C4.1, IC2.VDD, R9.1
- net +3V3: now also C4.1, IC2.REGIN, IC2.VDD, R9.1; no longer R1.1
- net +5V: no longer IC2.REGIN
- net GND: no longer C3.2
- net RESET: no longer C3.1, R1.2
Changed lines of the file:
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@@
 <part name="C1" library="SparkFun-Capacitors" library_urn="urn:adsk.eagle:library:510" deviceset="10UF" device="-0603-6.3V-20%" package3d_urn="urn:adsk.eagle:package:37414/1" value="10uF"/>
 <part name="C2" library="SparkFun-Capacitors" library_urn="urn:adsk.eagle:library:510" deviceset="10UF" device="-0603-6.3V-20%" package3d_urn="urn:adsk.eagle:package:37414/1" value="10uF"/>
-<part name="R1" library="RC0402FR-073M6L" deviceset="RC0402FR-073M6L" device="" value="100k"/>
-<part name="C3" library="SparkFun-Capacitors" deviceset="0.1UF" device="-0603-25V-(+80/-20%)" package3d_urn="urn:adsk.eagle:package:37414/1" value="0.1uF"/>
-<part name="GND8" library="supply1" library_urn="urn:adsk.eagle:library:371" deviceset="GND" device=""/>
 <part name="GND10" library="supply1" library_urn="urn:adsk.eagle:library:371" deviceset="GND" device=""/>
 <part name="GND11" library="supply1" library_urn="urn:adsk.eagle:library:371" deviceset="GND" device=""/>
@@
 <part name="R12" library="RC0402FR-073M6L" deviceset="RC0402FR-073M6L" device="" value="2.2k"/>
 <part name="D6" library="SparkFun-LED" library_urn="urn:adsk.eagle:library:529" deviceset="LED-BLUE" device="0603" package3d_urn="urn:adsk.eagle:package:39354/1" value="BLUE"/>
-<part name="P+5" library="supply1" library_urn="urn:adsk.eagle:library:371" deviceset="+5V" device=""/>
 <part name="P+6" library="supply1" library_urn="urn:adsk.eagle:library:371" deviceset="+5V" device=""/>
 <part name="J3" library="SparkFun-Connectors" library_urn="urn:adsk.eagle:library:513" deviceset="CORTEX_DEBUG" device="_SMD" package3d_urn="urn:adsk.eagle:package:38289/1"/>
@@
 <part name="PAD1" library="wirepad" library_urn="urn:adsk.eagle:library:412" deviceset="WIREPAD" device="SMD1,27-254" package3d_urn="urn:adsk.eagle:package:30839/1"/>
 <part name="PAD2" library="wirepad" library_urn="urn:adsk.eagle:library:412" deviceset="WIREPAD" device="SMD1,27-254" package3d_urn="urn:adsk.eagle:package:30839/1"/>
+<part name="+3V3" library="supply1" library_urn="urn:adsk.eagle:library:371" deviceset="+3V3" device=""/>
+<part name="P+5" library="supply1" library_urn="urn:adsk.eagle:library:371" deviceset="+5V" device=""/>
 </parts>
 <sheets>
@@
 <attribute name="VALUE" x="164.084" y="190.881" size="1.778" layer="96" font="vector"/>
 </instance>
-<instance part="R1" gate="G$1" x="99.06" y="45.72" smashed="yes" rot="R180">
-<attribute name="NAME" x="99.06" y="44.196" size="1.778" layer="95" font="vector" rot="R180" align="bottom-center"/>
-</instance>
-<instance part="C3" gate="G$1" x="86.36" y="27.94" smashed="yes">
-<attribute name="NAME" x="87.884" y="30.861" size="1.778" layer="95" font="vector"/>
-<attribute name="VALUE" x="87.884" y="25.781" size="1.778" layer="96" font="vector"/>
-</instance>
-<instance part="GND8" gate="1" x="86.36" y="20.32" smashed="yes">
-<attribute name="VALUE" x="83.82" y="17.78" size="1.778" layer="96"/>
-</instance>
 <instance part="GND10" gate="1" x="193.04" y="78.74" smashed="yes">
 <attribute name="VALUE" x="190.5" y="76.2" size="1.778" layer="96"/>
@@
 <attribute name="VALUE" x="191.135" y="182.372" size="1.778" layer="96" font="vector" rot="R270" align="top-left"/>
 </instance>
-<instance part="P+5" gate="1" x="35.56" y="157.48" smashed="yes">
-<attribute name="VALUE" x="33.02" y="152.4" size="1.778" layer="96" rot="R90"/>
-</instance>
 <instance part="P+6" gate="1" x="109.22" y="149.86" smashed="yes" rot="R270">
 <attribute name="VALUE" x="104.14" y="152.4" size="1.778" layer="96"/>
@@
 <instance part="PAD2" gate="G$1" x="233.68" y="195.58" smashed="yes" rot="R90">
 <attribute name="NAME" x="231.8258" y="194.437" size="1.778" layer="95" rot="R90"/>
+</instance>
+<instance part="+3V3" gate="G$1" x="35.56" y="157.48" smashed="yes">
+<attribute name="VALUE" x="33.02" y="152.4" size="1.778" layer="96" rot="R90"/>
+</instance>
+<instance part="P+5" gate="1" x="38.1" y="147.32" smashed="yes" rot="R90">
+<attribute name="VALUE" x="43.18" y="144.78" size="1.778" layer="96" rot="R180"/>
 </instance>
 </instances>
@@
 <net name="RESET" class="0">
 <segment>
-<pinref part="C3" gate="G$1" pin="1"/>
-<pinref part="R1" gate="G$1" pin="2"/>
-<wire x1="86.36" y1="45.72" x2="88.9" y2="45.72" width="0.1524" layer="91"/>
-<wire x1="86.36" y1="33.02" x2="86.36" y2="45.72" width="0.1524" layer="91"/>
-<junction x="86.36" y="45.72"/>
 <pinref part="U$1" gate="G$1" pin="RESET_N"/>
-<wire x1="71.12" y1="45.72" x2="86.36" y2="45.72" width="0.1524" layer="91"/>
+<wire x1="71.12" y1="45.72" x2="78.74" y2="45.72" width="0.1524" layer="91"/>
 <label x="71.12" y="45.72" size="1.778" layer="95"/>
 </segment>
@@
 <pinref part="C2" gate="G$1" pin="2"/>
 <wire x1="162.56" y1="190.5" x2="162.56" y2="185.42" width="0.1524" layer="91"/>
-</segment>
-<segment>
-<pinref part="C3" gate="G$1" pin="2"/>
-<wire x1="86.36" y1="25.4" x2="86.36" y2="22.86" width="0.1524" layer="91"/>
-<pinref part="GND8" gate="1" pin="GND"/>
 </segment>
 <segment>
@@
 </segment>
 </net>
-<net name="N$4" class="0">
-<segment>
-<pinref part="C4" gate="G$1" pin="1"/>
-<pinref part="R9" gate="G$1" pin="1"/>
-<wire x1="25.4" y1="144.78" x2="25.4" y2="142.24" width="0.1524" layer="91"/>
-<pinref part="IC2" gate="G$1" pin="VDD"/>
-<wire x1="25.4" y1="142.24" x2="43.18" y2="142.24" width="0.1524" layer="91"/>
-<junction x="25.4" y="142.24"/>
-</segment>
-</net>
 <net name="N$7" class="0">
 <segment>
@@
 </segment>
 <segment>
-<pinref part="IC2" gate="G$1" pin="VBUS"/>
-<wire x1="43.18" y1="147.32" x2="35.56" y2="147.32" width="0.1524" layer="91"/>
-<pinref part="IC2" gate="G$1" pin="REGIN"/>
-<wire x1="35.56" y1="147.32" x2="35.56" y2="149.86" width="0.1524" layer="91"/>
-<wire x1="35.56" y1="149.86" x2="43.18" y2="149.86" width="0.1524" layer="91"/>
-<wire x1="35.56" y1="149.86" x2="35.56" y2="154.94" width="0.1524" layer="91"/>
-<junction x="35.56" y="149.86"/>
-<pinref part="P+5" gate="1" pin="+5V"/>
-</segment>
-<segment>
 <pinref part="R8" gate="G$1" pin="2"/>
 <wire x1="104.14" y1="149.86" x2="106.68" y2="149.86" width="0.1524" layer="91"/>
@@
 <wire x1="93.98" y1="55.88" x2="101.6" y2="55.88" width="0.1524" layer="91"/>
 <pinref part="P+8" gate="1" pin="+5V"/>
+</segment>
+<segment>
+<pinref part="IC2" gate="G$1" pin="VBUS"/>
+<pinref part="P+5" gate="1" pin="+5V"/>
+<wire x1="40.64" y1="147.32" x2="43.18" y2="147.32" width="0.1524" layer="91"/>
 </segment>
 </net>
@@
 </segment>
 <segment>
-<pinref part="R1" gate="G$1" pin="1"/>
-<wire x1="109.22" y1="45.72" x2="116.84" y2="45.72" width="0.1524" layer="91"/>
-<label x="111.76" y="45.72" size="1.778" layer="95"/>
-</segment>
-<segment>
 <pinref part="U$1" gate="G$1" pin="VCC"/>
 <wire x1="45.72" y1="33.02" x2="45.72" y2="25.4" width="0.1524" layer="91"/>
@@
 <pinref part="+3V2" gate="G$1" pin="+3V3"/>
 </segment>
-</net>
+<segment>
+<pinref part="IC2" gate="G$1" pin="REGIN"/>
+<pinref part="+3V3" gate="G$1" pin="+3V3"/>
+<wire x1="43.18" y1="149.86" x2="35.56" y2="149.86" width="0.1524" layer="91"/>
+<wire x1="35.56" y1="149.86" x2="35.56" y2="154.94" width="0.1524" layer="91"/>
+<pinref part="C4" gate="G$1" pin="1"/>
+<pinref part="R9" gate="G$1" pin="1"/>
+<wire x1="25.4" y1="144.78" x2="25.4" y2="142.24" width="0.1524" layer="91"/>
+<pinref part="IC2" gate="G$1" pin="VDD"/>
+<wire x1="25.4" y1="142.24" x2="35.56" y2="142.24" width="0.1524" layer="91"/>
+<junction x="25.4" y="142.24"/>
+<wire x1="35.56" y1="142.24" x2="43.18" y2="142.24" width="0.1524" layer="91"/>
+<wire x1="35.56" y1="149.86" x2="35.56" y2="142.24" width="0.1524" layer="91"/>
+<junction x="35.56" y="149.86"/>
+<junction x="35.56" y="142.24"/>
+</segment>
+</net>

Commit message: Add files via upload
Parts:
- added C3: 100n, discretes-dev:CAP0402
- added R1: 2.2k, RC0402FR-073M6L:RC0402FR-073M6L
- added R15, R16: 0, RC0402FR-073M6L:RC0402FR-073M6L
- added U$2: MX25R8035FM1IL0, W25Q80BVSNIG:W25Q80BVSNIG
Connections:
- new net N$12: R15.2, U$2.HOLD/IO3
- new net N$15: R16.1, U$2.WP/IO2
- new net N$17: R1.2, U$2.CS
- net +3V3: now also C3.2, R1.1, R15.1, R16.2, U$2.VCC
- net DIO_10: now also U$2.CLK
- net DIO_8: now also U$2.DO/IO1
- net DIO_9: now also U$2.DI/IO0
- net GND: now also C3.1, U$2.GND
Other:
- moved on the sheet: CN1, D6, PAD1, PAD2, R11, R12, R2, U1, U3

Commit message: Add files via upload
Connections:
- removed net N$17: R1.2, U$2.CS
- net DIO_20: now also R1.2, U$2.CS
Other:
- moved on the sheet: R1
Changed lines of the file:
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@@
 </instance>
 <instance part="U$2" gate="G$1" x="238.76" y="58.42" smashed="yes"/>
-<instance part="R1" gate="G$1" x="274.32" y="55.88" smashed="yes" rot="R180">
-<attribute name="NAME" x="274.32" y="54.356" size="1.778" layer="95" font="vector" rot="R180" align="bottom-center"/>
+<instance part="R1" gate="G$1" x="279.4" y="55.88" smashed="yes" rot="R180">
+<attribute name="NAME" x="279.4" y="54.356" size="1.778" layer="95" font="vector" rot="R180" align="bottom-center"/>
 </instance>
 <instance part="C3" gate="G$1" x="215.9" y="50.8" smashed="yes" rot="R180">
@@
 <label x="116.84" y="66.04" size="1.778" layer="95"/>
 </segment>
+<segment>
+<pinref part="U$2" gate="G$1" pin="CS"/>
+<pinref part="R1" gate="G$1" pin="2"/>
+<wire x1="256.54" y1="55.88" x2="269.24" y2="55.88" width="0.1524" layer="91"/>
+<label x="259.08" y="55.88" size="1.778" layer="95"/>
+</segment>
 </net>
 <net name="DIO_21" class="0">
@@
 <segment>
 <pinref part="R1" gate="G$1" pin="1"/>
-<wire x1="284.48" y1="55.88" x2="287.02" y2="55.88" width="0.1524" layer="91"/>
-<wire x1="287.02" y1="55.88" x2="287.02" y2="63.5" width="0.1524" layer="91"/>
-<label x="287.02" y="58.42" size="1.778" layer="95" rot="R90"/>
+<wire x1="289.56" y1="55.88" x2="292.1" y2="55.88" width="0.1524" layer="91"/>
+<wire x1="292.1" y1="55.88" x2="292.1" y2="63.5" width="0.1524" layer="91"/>
+<label x="292.1" y="58.42" size="1.778" layer="95" rot="R90"/>
 </segment>
 <segment>
@@
 </segment>
 </net>
-<net name="N$17" class="0">
-<segment>
-<pinref part="U$2" gate="G$1" pin="CS"/>
-<pinref part="R1" gate="G$1" pin="2"/>
-<wire x1="256.54" y1="55.88" x2="264.16" y2="55.88" width="0.1524" layer="91"/>
-</segment>
-</net>
