File: cc2652p.sch (EAGLE design)
At the start: 44 parts, among them IC2 CP2102, J3 CORTEX_DEBUG_SMD, J5 TYPE-C-31-M-12, Q1 SI2323DS, U1 MCP73831, U2 ap2112k-3.3, U3 XC61CN3202MR-G

Commit message: Add files via upload
Parts:
- added C13: 220uF, Capacitor:C_TANTALUM-2917(7343-METRIC)
Connections:
- net +3V3: now also C13.1
- net GND: now also C13.2, J3.GNDDTCT; no longer J3.GND@3, J3.GND@5
Changed lines of the file:
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@@
 <part name="R15" library="RC0402FR-073M6L" deviceset="RC0402FR-073M6L" device="" value="0"/>
 <part name="R16" library="RC0402FR-073M6L" deviceset="RC0402FR-073M6L" device="" value="0"/>
+<part name="C13" library="Capacitor" library_urn="urn:adsk.eagle:library:16290819" deviceset="C" device="TANTALUM-2917(7343-METRIC)" package3d_urn="urn:adsk.eagle:package:16290891/2" technology="_" value="220uF"/>
 </parts>
 <sheets>
@@
 <attribute name="VALUE" x="124.46" y="205.74" size="1.778" layer="96"/>
 </instance>
-<instance part="+3V1" gate="G$1" x="172.72" y="198.12" smashed="yes" rot="R270">
-<attribute name="VALUE" x="167.64" y="200.66" size="1.778" layer="96"/>
+<instance part="+3V1" gate="G$1" x="182.88" y="198.12" smashed="yes" rot="R270">
+<attribute name="VALUE" x="177.8" y="200.66" size="1.778" layer="96"/>
 </instance>
 <instance part="P+1" gate="1" x="48.26" y="205.74" smashed="yes">
@@
 <attribute name="VALUE" x="152.4" y="48.514" size="1.778" layer="96" font="vector"/>
 </instance>
-<instance part="GND20" gate="1" x="142.24" y="55.88" smashed="yes">
-<attribute name="VALUE" x="139.7" y="53.34" size="1.778" layer="96"/>
+<instance part="GND20" gate="1" x="144.78" y="48.26" smashed="yes">
+<attribute name="VALUE" x="142.24" y="45.72" size="1.778" layer="96"/>
 </instance>
 <instance part="+3V4" gate="G$1" x="142.24" y="71.12" smashed="yes">
@@
 <instance part="R16" gate="G$1" x="251.46" y="73.66" smashed="yes" rot="R180">
 <attribute name="NAME" x="251.46" y="72.136" size="1.778" layer="95" font="vector" rot="R180" align="bottom-center"/>
+</instance>
+<instance part="C13" gate="G$1" x="172.72" y="195.58" smashed="yes">
+<attribute name="NAME" x="173.736" y="196.215" size="1.778" layer="95" font="vector"/>
+<attribute name="VALUE" x="173.736" y="191.389" size="1.778" layer="96" font="vector"/>
 </instance>
 </instances>
@@
 <pinref part="GND7" gate="1" pin="GND"/>
 <pinref part="C2" gate="G$1" pin="2"/>
-<wire x1="162.56" y1="190.5" x2="162.56" y2="185.42" width="0.1524" layer="91"/>
+<wire x1="162.56" y1="190.5" x2="162.56" y2="187.96" width="0.1524" layer="91"/>
+<pinref part="C13" gate="G$1" pin="2"/>
+<wire x1="162.56" y1="187.96" x2="162.56" y2="185.42" width="0.1524" layer="91"/>
+<wire x1="172.72" y1="190.5" x2="172.72" y2="187.96" width="0.1524" layer="91"/>
+<wire x1="172.72" y1="187.96" x2="162.56" y2="187.96" width="0.1524" layer="91"/>
+<junction x="162.56" y="187.96"/>
 </segment>
 <segment>
@@
 </segment>
 <segment>
-<pinref part="J3" gate="G$1" pin="GND@5"/>
-<wire x1="149.86" y1="58.42" x2="142.24" y2="58.42" width="0.1524" layer="91"/>
-<pinref part="J3" gate="G$1" pin="GND@3"/>
-<wire x1="149.86" y1="60.96" x2="142.24" y2="60.96" width="0.1524" layer="91"/>
-<wire x1="142.24" y1="58.42" x2="142.24" y2="60.96" width="0.1524" layer="91"/>
-<pinref part="GND20" gate="1" pin="GND"/>
-<junction x="142.24" y="58.42"/>
-</segment>
-<segment>
 <pinref part="U3" gate="A" pin="VSS"/>
 <wire x1="236.22" y1="124.46" x2="236.22" y2="121.92" width="0.1524" layer="91"/>
@@
 <pinref part="GND24" gate="1" pin="GND"/>
 <wire x1="261.62" y1="63.5" x2="261.62" y2="66.04" width="0.1524" layer="91"/>
+</segment>
+<segment>
+<pinref part="GND20" gate="1" pin="GND"/>
+<wire x1="144.78" y1="50.8" x2="144.78" y2="53.34" width="0.1524" layer="91"/>
+<pinref part="J3" gate="G$1" pin="GNDDTCT"/>
+<wire x1="144.78" y1="53.34" x2="149.86" y2="53.34" width="0.1524" layer="91"/>
 </segment>
 </net>
@@
 <wire x1="157.48" y1="198.12" x2="162.56" y2="198.12" width="0.1524" layer="91"/>
 <pinref part="C2" gate="G$1" pin="1"/>
-<wire x1="162.56" y1="198.12" x2="170.18" y2="198.12" width="0.1524" layer="91"/>
+<wire x1="162.56" y1="198.12" x2="172.72" y2="198.12" width="0.1524" layer="91"/>
 <junction x="162.56" y="198.12"/>
 <pinref part="+3V1" gate="G$1" pin="+3V3"/>
-</segment>
-<segment>
+<pinref part="C13" gate="G$1" pin="1"/>
+<wire x1="172.72" y1="198.12" x2="180.34" y2="198.12" width="0.1524" layer="91"/>
+<junction x="172.72" y="198.12"/>
+</segment>
+<segment>

Commit message: Add files via upload
Parts:
- added PSM: (no value), jumper:SJ
Connections:
- new net V+: C2.1, C4.1, IC2.REGIN, IC2.VDD, PSM.1, R9.1, U2.OUT
- net +3V3: now also PSM.2; no longer C2.1, C4.1, IC2.REGIN, IC2.VDD, R9.1, U2.OUT
Other:
- moved on the sheet: C13
Changed lines of the file:
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@@
 <part name="PAD1" library="wirepad" library_urn="urn:adsk.eagle:library:412" deviceset="WIREPAD" device="SMD1,27-254" package3d_urn="urn:adsk.eagle:package:30839/1"/>
 <part name="PAD2" library="wirepad" library_urn="urn:adsk.eagle:library:412" deviceset="WIREPAD" device="SMD1,27-254" package3d_urn="urn:adsk.eagle:package:30839/1"/>
-<part name="+3V3" library="supply1" library_urn="urn:adsk.eagle:library:371" deviceset="+3V3" device=""/>
 <part name="P+5" library="supply1" library_urn="urn:adsk.eagle:library:371" deviceset="+5V" device=""/>
 <part name="U$2" library="W25Q80BVSNIG" deviceset="W25Q80BVSNIG" device="" value="MX25R8035FM1IL0"/>
@@
 <part name="R16" library="RC0402FR-073M6L" deviceset="RC0402FR-073M6L" device="" value="0"/>
 <part name="C13" library="Capacitor" library_urn="urn:adsk.eagle:library:16290819" deviceset="C" device="TANTALUM-2917(7343-METRIC)" package3d_urn="urn:adsk.eagle:package:16290891/2" technology="_" value="220uF"/>
+<part name="PSM" library="jumper" library_urn="urn:adsk.eagle:library:252" deviceset="SJ" device="" package3d_urn="urn:adsk.eagle:package:15471/1"/>
+<part name="SUPPLY1" library="supply2" library_urn="urn:adsk.eagle:library:372" deviceset="V+" device="" value="3V3_USB"/>
+<part name="SUPPLY2" library="supply2" library_urn="urn:adsk.eagle:library:372" deviceset="V+" device="" value="3V3_USB"/>
 </parts>
 <sheets>
@@
 <attribute name="VALUE" x="124.46" y="205.74" size="1.778" layer="96"/>
 </instance>
-<instance part="+3V1" gate="G$1" x="182.88" y="198.12" smashed="yes" rot="R270">
-<attribute name="VALUE" x="177.8" y="200.66" size="1.778" layer="96"/>
+<instance part="+3V1" gate="G$1" x="187.96" y="198.12" smashed="yes" rot="R270">
+<attribute name="VALUE" x="182.88" y="200.66" size="1.778" layer="96"/>
 </instance>
 <instance part="P+1" gate="1" x="48.26" y="205.74" smashed="yes">
@@
 <attribute name="NAME" x="252.1458" y="194.437" size="1.778" layer="95" rot="R90"/>
 </instance>
-<instance part="+3V3" gate="G$1" x="35.56" y="157.48" smashed="yes">
-<attribute name="VALUE" x="33.02" y="152.4" size="1.778" layer="96" rot="R90"/>
-</instance>
 <instance part="P+5" gate="1" x="38.1" y="147.32" smashed="yes" rot="R90">
 <attribute name="VALUE" x="43.18" y="144.78" size="1.778" layer="96" rot="R180"/>
@@
 <attribute name="NAME" x="251.46" y="72.136" size="1.778" layer="95" font="vector" rot="R180" align="bottom-center"/>
 </instance>
-<instance part="C13" gate="G$1" x="172.72" y="195.58" smashed="yes">
-<attribute name="NAME" x="173.736" y="196.215" size="1.778" layer="95" font="vector"/>
-<attribute name="VALUE" x="173.736" y="191.389" size="1.778" layer="96" font="vector"/>
+<instance part="C13" gate="G$1" x="180.34" y="193.04" smashed="yes">
+<attribute name="NAME" x="181.356" y="193.675" size="1.778" layer="95" font="vector"/>
+<attribute name="VALUE" x="181.356" y="188.849" size="1.778" layer="96" font="vector"/>
+</instance>
+<instance part="PSM" gate="1" x="172.72" y="198.12" smashed="yes">
+<attribute name="NAME" x="170.18" y="200.66" size="1.778" layer="95"/>
+<attribute name="VALUE" x="170.18" y="194.31" size="1.778" layer="96"/>
+</instance>
+<instance part="SUPPLY1" gate="1" x="33.02" y="157.48" smashed="yes">
+<attribute name="VALUE" x="34.29" y="158.75" size="1.778" layer="96"/>
+</instance>
+<instance part="SUPPLY2" gate="1" x="162.56" y="205.74" smashed="yes">
+<attribute name="VALUE" x="163.83" y="207.01" size="1.778" layer="96"/>
 </instance>
 </instances>
@@
 <pinref part="C2" gate="G$1" pin="2"/>
 <wire x1="162.56" y1="190.5" x2="162.56" y2="187.96" width="0.1524" layer="91"/>
+<wire x1="162.56" y1="187.96" x2="162.56" y2="185.42" width="0.1524" layer="91"/>
+<wire x1="180.34" y1="187.96" x2="162.56" y2="187.96" width="0.1524" layer="91"/>
+<junction x="162.56" y="187.96"/>
 <pinref part="C13" gate="G$1" pin="2"/>
-<wire x1="162.56" y1="187.96" x2="162.56" y2="185.42" width="0.1524" layer="91"/>
-<wire x1="172.72" y1="190.5" x2="172.72" y2="187.96" width="0.1524" layer="91"/>
-<wire x1="172.72" y1="187.96" x2="162.56" y2="187.96" width="0.1524" layer="91"/>
-<junction x="162.56" y="187.96"/>
 </segment>
 <segment>
@@
 <net name="+3V3" class="0">
 <segment>
-<pinref part="U2" gate="G$1" pin="OUT"/>
-<wire x1="157.48" y1="198.12" x2="162.56" y2="198.12" width="0.1524" layer="91"/>
-<pinref part="C2" gate="G$1" pin="1"/>
-<wire x1="162.56" y1="198.12" x2="172.72" y2="198.12" width="0.1524" layer="91"/>
-<junction x="162.56" y="198.12"/>
-<pinref part="+3V1" gate="G$1" pin="+3V3"/>
-<pinref part="C13" gate="G$1" pin="1"/>
-<wire x1="172.72" y1="198.12" x2="180.34" y2="198.12" width="0.1524" layer="91"/>
-<junction x="172.72" y="198.12"/>
-</segment>
-<segment>
 <pinref part="U$1" gate="G$1" pin="VCC"/>
 <wire x1="45.72" y1="33.02" x2="45.72" y2="25.4" width="0.1524" layer="91"/>
@@
 <wire x1="93.98" y1="71.12" x2="101.6" y2="71.12" width="0.1524" layer="91"/>
 <pinref part="+3V2" gate="G$1" pin="+3V3"/>
-</segment>
-<segment>
-<pinref part="IC2" gate="G$1" pin="REGIN"/>
-<pinref part="+3V3" gate="G$1" pin="+3V3"/>
-<wire x1="43.18" y1="149.86" x2="35.56" y2="149.86" width="0.1524" layer="91"/>
-<wire x1="35.56" y1="149.86" x2="35.56" y2="154.94" width="0.1524" layer="91"/>
-<pinref part="C4" gate="G$1" pin="1"/>
-<pinref part="R9" gate="G$1" pin="1"/>
-<wire x1="25.4" y1="144.78" x2="25.4" y2="142.24" width="0.1524" layer="91"/>
-<pinref part="IC2" gate="G$1" pin="VDD"/>
-<wire x1="25.4" y1="142.24" x2="35.56" y2="142.24" width="0.1524" layer="91"/>
-<junction x="25.4" y="142.24"/>
-<wire x1="35.56" y1="142.24" x2="43.18" y2="142.24" width="0.1524" layer="91"/>
-<wire x1="35.56" y1="149.86" x2="35.56" y2="142.24" width="0.1524" layer="91"/>
-<junction x="35.56" y="149.86"/>
-<junction x="35.56" y="142.24"/>
 </segment>
 <segment>
@@
 <label x="238.76" y="78.74" size="1.778" layer="95" rot="R90"/>
 </segment>
+<segment>
+<pinref part="PSM" gate="1" pin="2"/>
+<wire x1="177.8" y1="198.12" x2="180.34" y2="198.12" width="0.1524" layer="91"/>
+<pinref part="C13" gate="G$1" pin="1"/>
+<wire x1="180.34" y1="198.12" x2="180.34" y2="195.58" width="0.1524" layer="91"/>
+<pinref part="+3V1" gate="G$1" pin="+3V3"/>
+<wire x1="180.34" y1="198.12" x2="185.42" y2="198.12" width="0.1524" layer="91"/>
+<junction x="180.34" y="198.12"/>
+</segment>
 </net>
 <net name="CC2" class="0">
@@
 </segment>
 </net>
+<net name="V+" class="0">
+<segment>
+<pinref part="C4" gate="G$1" pin="1"/>
+<pinref part="R9" gate="G$1" pin="1"/>
+<wire x1="25.4" y1="144.78" x2="25.4" y2="142.24" width="0.1524" layer="91"/>
+<pinref part="IC2" gate="G$1" pin="VDD"/>
+<wire x1="25.4" y1="142.24" x2="33.02" y2="142.24" width="0.1524" layer="91"/>
+<junction x="25.4" y="142.24"/>
+<pinref part="IC2" gate="G$1" pin="REGIN"/>
+<wire x1="33.02" y1="142.24" x2="43.18" y2="142.24" width="0.1524" layer="91"/>
+<wire x1="43.18" y1="149.86" x2="33.02" y2="149.86" width="0.1524" layer="91"/>
+<wire x1="33.02" y1="149.86" x2="33.02" y2="142.24" width="0.1524" layer="91"/>
+<junction x="33.02" y="142.24"/>
+<wire x1="33.02" y1="149.86" x2="33.02" y2="154.94" width="0.1524" layer="91"/>
+<junction x="33.02" y="149.86"/>
+<pinref part="SUPPLY1" gate="1" pin="V+"/>
+</segment>
+<segment>
+<pinref part="U2" gate="G$1" pin="OUT"/>
+<wire x1="157.48" y1="198.12" x2="162.56" y2="198.12" width="0.1524" layer="91"/>
+<pinref part="C2" gate="G$1" pin="1"/>
+<pinref part="PSM" gate="1" pin="1"/>
+<wire x1="162.56" y1="198.12" x2="167.64" y2="198.12" width="0.1524" layer="91"/>
+<junction x="162.56" y="198.12"/>
+<wire x1="162.56" y1="198.12" x2="162.56" y2="203.2" width="0.1524" layer="91"/>
+<pinref part="SUPPLY2" gate="1" pin="V+"/>
+</segment>
+</net>

Commit message: Add files via upload
Parts:
- removed PSM: (no value), jumper:SJ
- added Q2: SI2323DS, SI2323DS:SI2323DS
Connections:
- net +3V3: now also Q2.S; no longer PSM.2
- net GND: now also Q2.G
- net V+: now also Q2.D; no longer PSM.1
Changed lines of the file:
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@@
 <layer number="56" name="wert" color="7" fill="1" visible="no" active="no"/>
 <layer number="57" name="tCAD" color="7" fill="1" visible="no" active="no"/>
+<layer number="58" name="bCAD" color="7" fill="1" visible="no" active="no"/>
 <layer number="59" name="tCarbon" color="7" fill="1" visible="no" active="no"/>
 <layer number="60" name="bCarbon" color="7" fill="1" visible="no" active="no"/>
@@
 <layer number="136" name="silktop" color="7" fill="1" visible="yes" active="yes"/>
 <layer number="137" name="silkbottom" color="7" fill="1" visible="yes" active="yes"/>
+<layer number="138" name="mbTest" color="7" fill="1" visible="no" active="yes"/>
+<layer number="139" name="mtKeepout" color="7" fill="1" visible="no" active="yes"/>
+<layer number="140" name="mbKeepout" color="7" fill="1" visible="no" active="yes"/>
+<layer number="141" name="mtRestrict" color="7" fill="1" visible="no" active="yes"/>
+<layer number="142" name="mbRestrict" color="7" fill="1" visible="no" active="yes"/>
+<layer number="143" name="mvRestrict" color="7" fill="1" visible="no" active="yes"/>
 <layer number="144" name="Drill_legend" color="7" fill="1" visible="yes" active="yes"/>
 <layer number="145" name="DrillLegend_01-16" color="7" fill="1" visible="yes" active="yes"/>
 <layer number="146" name="DrillLegend_01-20" color="7" fill="1" visible="yes" active="yes"/>
+<layer number="147" name="mMeasures" color="7" fill="1" visible="no" active="yes"/>
+<layer number="148" name="mDocument" color="7" fill="1" visible="no" active="yes"/>
+<layer number="149" name="mReference" color="7" fill="1" visible="no" active="yes"/>
 <layer number="150" name="Notes" color="7" fill="1" visible="yes" active="yes"/>
 <layer number="151" name="HeatSink" color="7" fill="1" visible="yes" active="yes"/>
@@
 <layer number="154" name="FabDoc2" color="7" fill="1" visible="yes" active="yes"/>
 <layer number="155" name="FabDoc3" color="7" fill="1" visible="yes" active="yes"/>
+<layer number="156" name="V3OUTLINE" color="7" fill="1" visible="yes" active="yes"/>
 <layer number="166" name="AntennaArea" color="7" fill="1" visible="yes" active="yes"/>
 <layer number="168" name="4mmHeightArea" color="7" fill="1" visible="yes" active="yes"/>
 <layer number="188" name="188bmp" color="1" fill="10" visible="yes" active="yes"/>
+<layer number="191" name="mNets" color="7" fill="1" visible="no" active="yes"/>
+<layer number="192" name="mBusses" color="7" fill="1" visible="no" active="yes"/>
+<layer number="193" name="mPins" color="7" fill="1" visible="no" active="yes"/>
+<layer number="194" name="mSymbols" color="7" fill="1" visible="no" active="yes"/>
+<layer number="195" name="mNames" color="7" fill="1" visible="no" active="yes"/>
+<layer number="196" name="mValues" color="7" fill="1" visible="no" active="yes"/>
 <layer number="199" name="Contour" color="7" fill="1" visible="yes" active="yes"/>
 <layer number="200" name="200bmp" color="1" fill="10" visible="yes" active="yes"/>
@@
 <layer number="250" name="Descript" color="3" fill="1" visible="no" active="no"/>
 <layer number="251" name="SMDround" color="12" fill="11" visible="no" active="no"/>
+<layer number="253" name="DNP" color="62" fill="1" visible="yes" active="yes"/>
 <layer number="254" name="cooling" color="7" fill="1" visible="yes" active="yes"/>
 <layer number="255" name="routoute" color="7" fill="1" visible="yes" active="yes"/>
@@
 <part name="R16" library="RC0402FR-073M6L" deviceset="RC0402FR-073M6L" device="" value="0"/>
 <part name="C13" library="Capacitor" library_urn="urn:adsk.eagle:library:16290819" deviceset="C" device="TANTALUM-2917(7343-METRIC)" package3d_urn="urn:adsk.eagle:package:16290891/2" technology="_" value="220uF"/>
-<part name="PSM" library="jumper" library_urn="urn:adsk.eagle:library:252" deviceset="SJ" device="" package3d_urn="urn:adsk.eagle:package:15471/1"/>
 <part name="SUPPLY1" library="supply2" library_urn="urn:adsk.eagle:library:372" deviceset="V+" device="" value="3V3_USB"/>
 <part name="SUPPLY2" library="supply2" library_urn="urn:adsk.eagle:library:372" deviceset="V+" device="" value="3V3_USB"/>
+<part name="Q2" library="SI2323DS" deviceset="SI2323DS" device=""/>
 </parts>
 <sheets>
@@
 </instance>
 <instance part="Q1" gate="G$1" x="119.38" y="205.74" smashed="yes">
-<attribute name="NAME" x="124.46" y="208.28" size="1.778" layer="95"/>
-<attribute name="VALUE" x="124.46" y="205.74" size="1.778" layer="96"/>
+<attribute name="NAME" x="121.92" y="208.28" size="1.778" layer="95"/>
+<attribute name="VALUE" x="124.46" y="203.2" size="1.778" layer="96"/>
 </instance>
 <instance part="+3V1" gate="G$1" x="187.96" y="198.12" smashed="yes" rot="R270">
-<attribute name="VALUE" x="182.88" y="200.66" size="1.778" layer="96"/>
+<attribute name="VALUE" x="187.96" y="198.12" size="1.778" layer="96"/>
 </instance>
 <instance part="P+1" gate="1" x="48.26" y="205.74" smashed="yes">
@@
 <attribute name="VALUE" x="181.356" y="188.849" size="1.778" layer="96" font="vector"/>
 </instance>
-<instance part="PSM" gate="1" x="172.72" y="198.12" smashed="yes">
-<attribute name="NAME" x="170.18" y="200.66" size="1.778" layer="95"/>
-<attribute name="VALUE" x="170.18" y="194.31" size="1.778" layer="96"/>
-</instance>
 <instance part="SUPPLY1" gate="1" x="33.02" y="157.48" smashed="yes">
 <attribute name="VALUE" x="34.29" y="158.75" size="1.778" layer="96"/>
@@
 <instance part="SUPPLY2" gate="1" x="162.56" y="205.74" smashed="yes">
 <attribute name="VALUE" x="163.83" y="207.01" size="1.778" layer="96"/>
+</instance>
+<instance part="Q2" gate="G$1" x="172.72" y="198.12" smashed="yes" rot="R90">
+<attribute name="VALUE" x="175.26383125" y="200.66383125" size="1.78068125" layer="96"/>
+<attribute name="NAME" x="170.18" y="200.662209375" size="1.77955" layer="95"/>
 </instance>
 </instances>
@@
 <wire x1="162.56" y1="190.5" x2="162.56" y2="187.96" width="0.1524" layer="91"/>
 <wire x1="162.56" y1="187.96" x2="162.56" y2="185.42" width="0.1524" layer="91"/>
-<wire x1="180.34" y1="187.96" x2="162.56" y2="187.96" width="0.1524" layer="91"/>
+<wire x1="180.34" y1="187.96" x2="175.26" y2="187.96" width="0.1524" layer="91"/>
 <junction x="162.56" y="187.96"/>
 <pinref part="C13" gate="G$1" pin="2"/>
+<pinref part="Q2" gate="G$1" pin="G"/>
+<wire x1="175.26" y1="187.96" x2="162.56" y2="187.96" width="0.1524" layer="91"/>
+<wire x1="175.26" y1="193.04" x2="175.26" y2="187.96" width="0.1524" layer="91"/>
+<junction x="175.26" y="187.96"/>
 </segment>
 <segment>
@@
 </segment>
 <segment>
-<pinref part="PSM" gate="1" pin="2"/>
 <wire x1="177.8" y1="198.12" x2="180.34" y2="198.12" width="0.1524" layer="91"/>
 <pinref part="C13" gate="G$1" pin="1"/>
@@
 <wire x1="180.34" y1="198.12" x2="185.42" y2="198.12" width="0.1524" layer="91"/>
 <junction x="180.34" y="198.12"/>
+<pinref part="Q2" gate="G$1" pin="S"/>
 </segment>
 </net>
@@
 <wire x1="157.48" y1="198.12" x2="162.56" y2="198.12" width="0.1524" layer="91"/>
 <pinref part="C2" gate="G$1" pin="1"/>
-<pinref part="PSM" gate="1" pin="1"/>
 <wire x1="162.56" y1="198.12" x2="167.64" y2="198.12" width="0.1524" layer="91"/>
 <junction x="162.56" y="198.12"/>
 <wire x1="162.56" y1="198.12" x2="162.56" y2="203.2" width="0.1524" layer="91"/>
 <pinref part="SUPPLY2" gate="1" pin="V+"/>
-</segment>
-</net>
+<pinref part="Q2" gate="G$1" pin="D"/>
+</segment>
+</net>

Commit message: Add files via upload
Parts:
- removed Q2: SI2323DS, SI2323DS:SI2323DS
- added PSM: PSM, pimoroni-misc:SOLDER_JUMPER_CLOSED
Connections:
- net +3V3: now also PSM.2; no longer Q2.S
- net GND: no longer Q2.G
- net V+: now also PSM.1; no longer Q2.D
Changed lines of the file:
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@@
 <part name="SUPPLY1" library="supply2" library_urn="urn:adsk.eagle:library:372" deviceset="V+" device="" value="3V3_USB"/>
 <part name="SUPPLY2" library="supply2" library_urn="urn:adsk.eagle:library:372" deviceset="V+" device="" value="3V3_USB"/>
-<part name="Q2" library="SI2323DS" deviceset="SI2323DS" device=""/>
+<part name="PSM" library="pimoroni-misc" deviceset="SOLDER_JUMPER_CLOSED" device="" value="PSM"/>
 </parts>
 <sheets>
@@
 <attribute name="VALUE" x="163.83" y="207.01" size="1.778" layer="96"/>
 </instance>
-<instance part="Q2" gate="G$1" x="172.72" y="198.12" smashed="yes" rot="R90">
-<attribute name="VALUE" x="175.26383125" y="200.66383125" size="1.78068125" layer="96"/>
-<attribute name="NAME" x="170.18" y="200.662209375" size="1.77955" layer="95"/>
-</instance>
+<instance part="PSM" gate="G$1" x="172.72" y="198.12" smashed="yes"/>
 </instances>
 <busses>
@@
 <wire x1="162.56" y1="190.5" x2="162.56" y2="187.96" width="0.1524" layer="91"/>
 <wire x1="162.56" y1="187.96" x2="162.56" y2="185.42" width="0.1524" layer="91"/>
-<wire x1="180.34" y1="187.96" x2="175.26" y2="187.96" width="0.1524" layer="91"/>
 <junction x="162.56" y="187.96"/>
 <pinref part="C13" gate="G$1" pin="2"/>
-<pinref part="Q2" gate="G$1" pin="G"/>
-<wire x1="175.26" y1="187.96" x2="162.56" y2="187.96" width="0.1524" layer="91"/>
-<wire x1="175.26" y1="193.04" x2="175.26" y2="187.96" width="0.1524" layer="91"/>
-<junction x="175.26" y="187.96"/>
+<wire x1="180.34" y1="187.96" x2="162.56" y2="187.96" width="0.1524" layer="91"/>
 </segment>
 <segment>
@@
 </segment>
 <segment>
-<wire x1="177.8" y1="198.12" x2="180.34" y2="198.12" width="0.1524" layer="91"/>
 <pinref part="C13" gate="G$1" pin="1"/>
 <wire x1="180.34" y1="198.12" x2="180.34" y2="195.58" width="0.1524" layer="91"/>
@@
 <wire x1="180.34" y1="198.12" x2="185.42" y2="198.12" width="0.1524" layer="91"/>
 <junction x="180.34" y="198.12"/>
-<pinref part="Q2" gate="G$1" pin="S"/>
+<pinref part="PSM" gate="G$1" pin="2"/>
+<wire x1="175.26" y1="198.12" x2="180.34" y2="198.12" width="0.1524" layer="91"/>
 </segment>
 </net>
@@
 <wire x1="157.48" y1="198.12" x2="162.56" y2="198.12" width="0.1524" layer="91"/>
 <pinref part="C2" gate="G$1" pin="1"/>
-<wire x1="162.56" y1="198.12" x2="167.64" y2="198.12" width="0.1524" layer="91"/>
+<wire x1="162.56" y1="198.12" x2="170.18" y2="198.12" width="0.1524" layer="91"/>
 <junction x="162.56" y="198.12"/>
 <wire x1="162.56" y1="198.12" x2="162.56" y2="203.2" width="0.1524" layer="91"/>
 <pinref part="SUPPLY2" gate="1" pin="V+"/>
-<pinref part="Q2" gate="G$1" pin="D"/>
-</segment>
-</net>
+<pinref part="PSM" gate="G$1" pin="1"/>
+</segment>
+</net>
