File: cc2652p.sch (EAGLE design)
At the start: 46 parts, among them IC2 CP2102, J3 CORTEX_DEBUG_SMD, J5 TYPE-C-31-M-12, Q1 SI2323DS, U1 MCP73831, U2 ap2112k-3.3, U3 XC61CN3202MR-G

Commit message: Add files via upload
Parts:
- removed PSM: PSM, pimoroni-misc:SOLDER_JUMPER_CLOSED
- added Q2: SI2323DS, SI2323DS:SI2323DS
- added R17, R18: 100k, RC0402FR-073M6L:RC0402FR-073M6L
- added SJ1: PSM, pimoroni-misc:SMALL_SOLDER_JUMPER_CLOSED
- added U4: MMDT2907A-7-F, MMDT2907A-7-F:MMDT2907A-7-F
Connections:
- new net N$10: Q2.G, R17.2, U4.C2
- new net N$4: R18.2, U4.B1, U4.B2, U4.C1
- net +3V3: now also Q2.S, SJ1.2, U4.E2; no longer PSM.2
- net GND: now also R17.1, R18.1
- net V+: now also Q2.D, SJ1.1, U4.E1; no longer PSM.1
Other:
- moved on the sheet: C13, CN1, D6, PAD1, PAD2, R1, R11, R12, R2, U1, U3

Commit message: Add files via upload
Parts:
- added U5: MX25R8035FZUIL0, MX25R8035FZUIL0:MX25R8035FZUIL0
- D5: value (none) -> MBR0540
Connections:
- net +3V3: now also U5.VCC
- net DIO_10: now also U5.SCLK
- net DIO_20: now also U5.!CS
- net DIO_8: now also U5.SO/SIO1
- net DIO_9: now also U5.SI/SIO0
- net GND: now also U5.EXP, U5.GND
- net N$12: now also U5.!RESET!/SIO3
- net N$15: now also U5.!WP!/SIO2
Other:
- moved on the sheet: C3, R1, R15, R16

Commit message: Add files via upload
Parts:
- R1: value 2.2k -> 100k
- R15, R16: value 0 -> 10k
- U5: value MX25R8035FZUIL0 -> W25X40CL
Changed lines of the file:
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@@
 <part name="P+5" library="supply1" library_urn="urn:adsk.eagle:library:371" deviceset="+5V" device=""/>
 <part name="U$2" library="W25Q80BVSNIG" deviceset="W25Q80BVSNIG" device="" value="MX25R8035FM1IL0"/>
-<part name="R1" library="RC0402FR-073M6L" deviceset="RC0402FR-073M6L" device="" value="2.2k"/>
+<part name="R1" library="RC0402FR-073M6L" deviceset="RC0402FR-073M6L" device="" value="100k"/>
 <part name="C3" library="discretes-dev" deviceset="CAP0402" device="" value="100n"/>
 <part name="GND8" library="supply1" library_urn="urn:adsk.eagle:library:371" deviceset="GND" device=""/>
 <part name="GND24" library="supply1" library_urn="urn:adsk.eagle:library:371" deviceset="GND" device=""/>
-<part name="R15" library="RC0402FR-073M6L" deviceset="RC0402FR-073M6L" device="" value="0"/>
-<part name="R16" library="RC0402FR-073M6L" deviceset="RC0402FR-073M6L" device="" value="0"/>
+<part name="R15" library="RC0402FR-073M6L" deviceset="RC0402FR-073M6L" device="" value="10k"/>
+<part name="R16" library="RC0402FR-073M6L" deviceset="RC0402FR-073M6L" device="" value="10k"/>
 <part name="C13" library="Capacitor" library_urn="urn:adsk.eagle:library:16290819" deviceset="C" device="TANTALUM-2917(7343-METRIC)" package3d_urn="urn:adsk.eagle:package:16290891/2" technology="_" value="220uF"/>
 <part name="SUPPLY1" library="supply2" library_urn="urn:adsk.eagle:library:372" deviceset="V+" device="" value="3V3_USB"/>
@@
 <part name="GND28" library="supply1" library_urn="urn:adsk.eagle:library:371" deviceset="GND" device=""/>
 <part name="SJ1" library="pimoroni-misc" deviceset="SMALL_SOLDER_JUMPER_CLOSED" device="" value="PSM"/>
-<part name="U5" library="MX25R8035FZUIL0" deviceset="MX25R8035FZUIL0" device=""/>
+<part name="U5" library="MX25R8035FZUIL0" deviceset="MX25R8035FZUIL0" device="" value="W25X40CL"/>
 <part name="GND29" library="supply1" library_urn="urn:adsk.eagle:library:371" deviceset="GND" device=""/>
 </parts>
