File: RF-BM-2652P2/cc2652p_rf-star.brd (EAGLE design)
At the start: 25.3 x 57.3 mm, 41 parts, among them IC2 CP2102, J3 CORTEX_DEBUG_SMD, J5 TYPE-C-31-M-12, Q1 SI2323DS, U1 MCP73831, U2 ap2112k-3.3, U3 XC61CN3202MR-G

Commit message: Add files via upload
Parts:
- moved R1 2.79 mm to (12.8, 18.9), turned to 180 degrees
- moved C3 1.85 mm to (12.2, 20.3), turned to 180 degrees
Routing:
- net GND: track 22.0 -> 19.8 mm, vias 97 -> 98
- net RES: track 41.6 -> 41.0 mm
- net +3V3: track 60.4 -> 60.1 mm, vias 3 -> 2

Commit message: Add files via upload
Connections:
- net RES: now also J3.10
Routing:
- net +5V: track 56.8 -> 63.6 mm, vias 4 -> 5
- net VCC: track 47.7 -> 52.2 mm
- net RES: track 41.0 -> 43.0 mm
- net 18: track 12.4 -> 13.2 mm
- net GND: track 19.8 -> 20.1 mm, vias 98 -> 99

Commit message: Add files via upload
Parts:
- moved R3 0.57 mm to (1.19, 50.5)
- moved R5 0.46 mm to (23.7, 50.5)
Routing:
- net DTR: track 11.3 -> 6.99 mm
- net GND: track 20.1 -> 17.1 mm, vias 99 -> 97
- net 7: track 14.8 -> 17.4 mm, vias 1 -> 0
- net 6: track 32.3 -> 30.2 mm
- net +3V3: track 59.9 -> 58.8 mm
- net 15: track 41.9 -> 42.6 mm

Commit message: Add files via upload
Parts:
- moved D2 0.38 mm to (22.8, 51.7)
- moved D1 0.38 mm to (2.13, 51.7)
Other:
- outline, holes or cut-outs redrawn
Changed lines of the file:
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@@
 <drawing>
 <settings>
-<setting alwaysvectorfont="yes"/>
+<setting alwaysvectorfont="no"/>
 <setting verticaltext="up"/>
 </settings>
@@
 <wire x1="2.1" y1="57.2" x2="2.2" y2="57.2" width="0.0762" layer="20"/>
 <wire x1="-0.2" y1="55.2" x2="2.2" y2="57.2" width="0.0762" layer="20" curve="-87.473883"/>
-<wire x1="2.2" y1="57.2" x2="3.7" y2="57.2" width="0.0762" layer="20"/>
-<wire x1="3.7" y1="57.2" x2="3.7" y2="51.2" width="0.0762" layer="20"/>
-<wire x1="3.7" y1="51.2" x2="21.3" y2="51.2" width="0.0762" layer="20"/>
-<wire x1="21.3" y1="51.2" x2="21.3" y2="57.2" width="0.0762" layer="20"/>
-<wire x1="21.3" y1="57.2" x2="22.7" y2="57.2" width="0.0762" layer="20"/>
+<wire x1="2.2" y1="57.2" x2="4.081" y2="57.2" width="0.0762" layer="20"/>
+<wire x1="4.081" y1="57.2" x2="4.081" y2="51.2" width="0.0762" layer="20"/>
+<wire x1="4.081" y1="51.2" x2="20.919" y2="51.2" width="0.0762" layer="20"/>
+<wire x1="20.919" y1="51.2" x2="20.919" y2="57.2" width="0.0762" layer="20"/>
+<wire x1="20.919" y1="57.2" x2="22.7" y2="57.2" width="0.0762" layer="20"/>
 <wire x1="22.7" y1="57.2" x2="22.8" y2="57.2" width="0.0762" layer="20"/>
 <wire x1="-0.2" y1="55.2" x2="-0.2" y2="2.3" width="0.0762" layer="20"/>
@@
 <text x="2.94" y="9.86" size="0.8128" layer="25" font="vector" ratio="12" rot="R90">5V</text>
 <text x="12.9" y="0.3" size="0.8128" layer="25" font="vector" ratio="12" rot="R90">PWR</text>
-<text x="1.546" y="52.327" size="0.8128" layer="25" font="vector" ratio="12">R</text>
-<text x="23.027" y="52.327" size="0.8128" layer="25" font="vector" ratio="12">G</text>
+<text x="1.927" y="52.454" size="0.8128" layer="25" font="vector" ratio="12">R</text>
+<text x="22.646" y="52.454" size="0.8128" layer="25" font="vector" ratio="12">G</text>
 <text x="14.3" y="0.3" size="0.8128" layer="25" font="vector" ratio="12" rot="R90">CHG</text>
 <text x="2.9" y="38.281" size="0.8128" layer="25" font="vector" ratio="12" rot="R90">9</text>
@@
 <attribute name="VALUE" x="17.724" y="23.6" size="0.6096" layer="27" font="vector" ratio="20" rot="R90" align="top-center"/>
 </element>
-<element name="D1" library="SparkFun-LED" library_urn="urn:adsk.eagle:library:529" package="LED-0603" package3d_urn="urn:adsk.eagle:package:39354/1" value="RED" x="1.746" y="51.654" smashed="yes" rot="R180">
-<attribute name="PROD_ID" value="DIO-00819" x="1.446" y="48.354" size="1.778" layer="27" rot="R180" display="off"/>
-</element>
-<element name="D2" library="SparkFun-LED" library_urn="urn:adsk.eagle:library:529" package="LED-0603" package3d_urn="urn:adsk.eagle:package:39354/1" value="GREEN" x="23.227" y="51.654" smashed="yes">
-<attribute name="PROD_ID" value="DIO-00821" x="23.527" y="54.954" size="1.778" layer="27" display="off"/>
+<element name="D1" library="SparkFun-LED" library_urn="urn:adsk.eagle:library:529" package="LED-0603" package3d_urn="urn:adsk.eagle:package:39354/1" value="RED" x="2.127" y="51.654" smashed="yes" rot="R180">
+<attribute name="PROD_ID" value="DIO-00819" x="1.827" y="48.354" size="1.778" layer="27" rot="R180" display="off"/>
+</element>
+<element name="D2" library="SparkFun-LED" library_urn="urn:adsk.eagle:library:529" package="LED-0603" package3d_urn="urn:adsk.eagle:package:39354/1" value="GREEN" x="22.846" y="51.654" smashed="yes">
+<attribute name="PROD_ID" value="DIO-00821" x="23.146" y="54.954" size="1.778" layer="27" display="off"/>
 </element>
 <element name="R5" library="RC0402FR-073M6L" package="RESC1005X40N" value="2.2k" x="23.708" y="50.454" smashed="yes">
@@
 <contactref element="D1" pad="C"/>
 <contactref element="R3" pad="2"/>
-<wire x1="0.869" y1="51.654" x2="0.869" y2="50.563" width="0.2" layer="1"/>
-<wire x1="0.76" y1="50.454" x2="0.869" y2="50.563" width="0.2" layer="1"/>
+<wire x1="1.25" y1="51.654" x2="1.25" y2="51.198" width="0.2" layer="1"/>
+<wire x1="1.25" y1="51.198" x2="0.76" y2="50.708" width="0.2" layer="1"/>
+<wire x1="0.76" y1="50.454" x2="0.76" y2="50.708" width="0.2" layer="1"/>
 </signal>
 <signal name="N$3">
 <contactref element="D2" pad="C"/>
 <contactref element="R5" pad="2"/>
-<wire x1="24.104" y1="51.654" x2="24.104" y2="50.49" width="0.2" layer="1"/>
-<wire x1="24.14" y1="50.454" x2="24.104" y2="50.49" width="0.2" layer="1"/>
+<wire x1="23.723" y1="51.654" x2="23.723" y2="51.125" width="0.2" layer="1"/>
+<wire x1="24.14" y1="50.454" x2="24.14" y2="50.708" width="0.2" layer="1"/>
+<wire x1="24.14" y1="50.708" x2="23.723" y2="51.125" width="0.2" layer="1"/>
 </signal>
 <signal name="D+">
@@
 <wire x1="13.208" y1="23.876" x2="13.208" y2="23.749" width="0.2" layer="16"/>
 <wire x1="4.245" y1="33.658" x2="6.337375" y2="33.658" width="0.254" layer="1"/>
-<wire x1="6.337375" y1="33.658" x2="7.9994" y2="31.995975" width="0.254" layer="1"/>
+<wire x1="6.337375" y1="33.658" x2="7.7421875" y2="32.2531875" width="0.254" layer="1"/>
+<wire x1="7.7421875" y1="32.2531875" x2="7.9994" y2="31.995975" width="0.254" layer="1"/>
 <wire x1="7.9994" y1="31.995975" x2="7.9994" y2="28.448" width="0.254" layer="1"/>
 <wire x1="8.382" y1="28.067" x2="12.192" y2="28.067" width="0.254" layer="16"/>
@@
 <contactref element="D1" pad="A"/>
 <wire x1="3.813" y1="42.545" x2="3.81" y2="42.548" width="0.2" layer="1"/>
-<wire x1="2.623" y1="51.654" x2="2.667" y2="51.61" width="0.2" layer="1"/>
-<wire x1="2.667" y1="50.292" x2="3.81" y2="49.149" width="0.2" layer="1"/>
+<wire x1="3.048" y1="49.911" x2="3.81" y2="49.149" width="0.2" layer="1"/>
 <wire x1="3.81" y1="49.149" x2="3.81" y2="46.482" width="0.2" layer="1"/>
 <wire x1="3.81" y1="46.482" x2="4.318" y2="45.974" width="0.2" layer="1"/>
@@
 <wire x1="6.477" y1="43.053" x2="5.972" y2="42.548" width="0.2" layer="1"/>
 <wire x1="5.972" y1="42.548" x2="4.245" y2="42.548" width="0.2" layer="1"/>
-<wire x1="2.667" y1="51.61" x2="2.667" y2="50.292" width="0.2" layer="1"/>
+<wire x1="3.004" y1="51.654" x2="3.048" y2="51.61" width="0.2" layer="1"/>
+<wire x1="3.048" y1="51.61" x2="3.048" y2="49.911" width="0.2" layer="1"/>
 <wire x1="4.318" y1="45.974" x2="5.842" y2="45.974" width="0.2" layer="1"/>
 </signal>
@@
 <wire x1="1.474625" y1="46.16" x2="2.667" y2="44.967625" width="0.2" layer="1"/>
 <contactref element="D2" pad="A"/>
-<wire x1="22.35" y1="51.654" x2="22.352" y2="51.652" width="0.2" layer="1"/>
-<wire x1="22.352" y1="51.652" x2="22.352" y2="50.546" width="0.2" layer="1"/>
+<wire x1="21.969" y1="51.654" x2="21.971" y2="51.652" width="0.2" layer="1"/>
+<wire x1="21.971" y1="51.652" x2="21.971" y2="50.927" width="0.2" layer="1"/>
+<wire x1="21.971" y1="50.927" x2="22.352" y2="50.546" width="0.2" layer="1"/>
 <via x="22.352" y="50.546" extent="1-16" drill="0.3"/>
 <wire x1="22.479" y1="50.419" x2="22.352" y2="50.546" width="0.2" layer="16"/>

Commit message: Add files via upload
RX TX fix
Connections:
- removed net DIO_12: IC2.26
- removed net DIO_13: IC2.25
- net 12: now also IC2.26
- net 13: now also IC2.25
Routing:
- net 12: track 7.40 -> 36.0 mm, vias 0 -> 2
- net 13: track 8.66 -> 34.4 mm, vias 0 -> 2
- net +3V3: track 58.8 -> 75.1 mm
- net +5V: track 64.0 -> 54.8 mm, vias 5 -> 4
- net VCC: track 52.2 -> 55.8 mm
- net DTR: track 6.99 -> 8.64 mm
- net TDI: track 34.2 -> 35.3 mm
- net TDO: track 31.4 -> 30.4 mm
- net GND: vias 97 -> 91
Other:
- board text added: "DIO10"
- board text added: "DIO11"
- board text added: "DIO12"
- board text added: "DIO13"
- board text added: "DIO14"
- board text added: "DIO15"
- board text added: "DIO18"
- board text added: "DIO19"
- board text added: "DIO20"
- board text added: "DIO21"
- board text added: "DIO22"
- board text added: "DIO23"
- board text added: "DIO24"
- board text added: "DIO25"
- board text added: "DIO26"
- board text added: "DIO27"
- board text added: "DIO5"
- board text added: "DIO6"
- board text added: "DIO7"
- board text added: "DIO8"
- board text added: "DIO9"

Commit message: Add files via upload
Parts:
- removed C3: 0.1uF, SparkFun-Capacitors:0603
- removed R1: 100k, RC0402FR-073M6L:RESC1005X40N
Connections:
- removed net N$4: C4.1, IC2.6, R9.1
- net +3V3: now also C4.1, IC2.6, IC2.7, R9.1; no longer R1.1
- net +5V: no longer IC2.7
- net GND: no longer C3.2
- net RES: no longer C3.1, R1.2
Routing:
- net N$4: track 6.86 -> 0.00 mm
- net +3V3: track 75.1 -> 81.4 mm, vias 2 -> 3
- net RES: track 43.3 -> 41.2 mm
- net VCC: track 55.8 -> 57.2 mm
- net +5V: track 54.8 -> 55.0 mm, vias 4 -> 3
- net GND: vias 91 -> 94

Commit message: Add files via upload
Parts:
- added C3: 100n, discretes-dev:CAPC1005X40N
- added R1: 2.2k, RC0402FR-073M6L:RESC1005X40N
- added R15, R16: 0, RC0402FR-073M6L:RESC1005X40N
- added U$1: MX25R8035FM1IL0, W25Q80BVSNIG:SO-8
Connections:
- new net N$12: R15.2, U$1.7
- new net N$15: R16.1, U$1.3
- new net N$17: R1.2, U$1.1
- net +3V3: now also C3.2, R1.1, R15.1, R16.2, U$1.8
- net 10: now also U$1.6
- net 8: now also U$1.2
- net 9: now also U$1.5
- net GND: now also C3.1, U$1.4
Routing:
- net +3V3: track 81.4 -> 104.5 mm
- net 8: track 3.33 -> 18.6 mm, vias 0 -> 1
- net N$15: track 0.00 -> 9.71 mm
- net 9: track 4.11 -> 13.5 mm, vias 0 -> 1
- net N$12: track 0.00 -> 6.43 mm
- net 10: track 5.06 -> 10.1 mm, vias 0 -> 1
- net N$17: track 0.00 -> 1.40 mm
- net 6: track 30.4 -> 29.8 mm
- net GND: vias 94 -> 88

Commit message: Add files via upload
Connections:
- removed net N$17: R1.2, U$1.1
- net 20: now also R1.2, U$1.1
Routing:
- net 20: track 7.38 -> 23.7 mm, vias 0 -> 1
- net N$17: track 1.40 -> 0.00 mm
- net GND: vias 88 -> 81
Changed lines of the file:
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@@
 <drawing>
 <settings>
-<setting alwaysvectorfont="no"/>
+<setting alwaysvectorfont="yes"/>
 <setting verticaltext="up"/>
 </settings>
@@
 <via x="7.468" y="36.565" extent="1-16" drill="0.3"/>
 <via x="10.008" y="36.565" extent="1-16" drill="0.3"/>
-<via x="12.548" y="36.565" extent="1-16" drill="0.3"/>
-<via x="15.088" y="36.565" extent="1-16" drill="0.3"/>
-<via x="17.628" y="36.565" extent="1-16" drill="0.3"/>
 <via x="10.008" y="34.025" extent="1-16" drill="0.3"/>
-<via x="12.548" y="34.025" extent="1-16" drill="0.3"/>
 <via x="15.088" y="34.025" extent="1-16" drill="0.3"/>
 <via x="17.628" y="34.025" extent="1-16" drill="0.3"/>
-<via x="10.008" y="31.485" extent="1-16" drill="0.3"/>
-<via x="12.548" y="39.105" extent="1-16" drill="0.3"/>
 <via x="12.548" y="44.185" extent="1-16" drill="0.3"/>
-<via x="12.548" y="28.945" extent="1-16" drill="0.3"/>
 </signal>
 <signal name="VCC">
@@
 <via x="5.588" y="29.845" extent="1-16" drill="0.3"/>
 <wire x1="4.245" y1="29.848" x2="5.585" y2="29.848" width="0.508" layer="1"/>
-<wire x1="5.588" y1="29.845" x2="13.716" y2="29.845" width="0.508" layer="16"/>
-<wire x1="13.716" y1="29.845" x2="17.145" y2="26.416" width="0.508" layer="16"/>
-<wire x1="17.145" y1="26.416" x2="17.145" y2="20.2" width="0.508" layer="16"/>
+<wire x1="17.145" y1="20.2" x2="17.145" y2="26.924" width="0.508" layer="16"/>
 <wire x1="17.1" y1="20.2" x2="17.1" y2="20.111" width="0.508" layer="16"/>
 <wire x1="18.991" y1="18.22" x2="23.9" y2="18.22" width="0.508" layer="16"/>
@@
 <wire x1="8.9408" y1="43.5358" x2="8.966" y2="43.561" width="0.2" layer="16"/>
 <wire x1="14.804665625" y1="44.69640625" x2="14.8298875" y2="44.721628125" width="0.2" layer="16"/>
-<wire x1="13.716" y1="43.053" x2="14.224" y2="43.561" width="0.508" layer="16"/>
+<wire x1="14.224" y1="43.561" x2="12.827" y2="42.164" width="0.508" layer="16"/>
 <wire x1="14.224" y1="43.561" x2="14.8298875" y2="43.561" width="0.508" layer="16"/>
-<wire x1="13.716" y1="29.845" x2="13.716" y2="42.164" width="0.508" layer="16"/>
-<wire x1="13.716" y1="42.164" x2="13.716" y2="43.053" width="0.508" layer="16"/>
-<wire x1="8.9408" y1="42.164" x2="13.716" y2="42.164" width="0.508" layer="16"/>
+<wire x1="8.9408" y1="42.164" x2="12.827" y2="42.164" width="0.508" layer="16"/>
+<wire x1="12.827" y1="42.164" x2="12.827" y2="31.242" width="0.508" layer="16"/>
+<wire x1="17.145" y1="26.924" x2="12.827" y2="31.242" width="0.508" layer="16"/>
+<wire x1="12.827" y1="31.242" x2="6.985" y2="31.242" width="0.508" layer="16"/>
+<wire x1="6.985" y1="31.242" x2="5.588" y2="29.845" width="0.508" layer="16"/>
 </signal>
 <signal name="CC2">
@@
 <wire x1="22.7078" y1="35.00779375" x2="22.7078" y2="32.9182" width="0.2" layer="1"/>
 <wire x1="22.7078" y1="32.9182" x2="23.9" y2="31.726" width="0.2" layer="1"/>
+<contactref element="U$1" pad="1"/>
+<contactref element="R1" pad="2"/>
+<wire x1="15.6938875" y1="43.561" x2="15.6972" y2="43.5576875" width="0.2" layer="16"/>
+<wire x1="15.6972" y1="43.5576875" x2="15.6972" y2="42.164" width="0.2" layer="16"/>
+<wire x1="15.6972" y1="42.164" x2="13.843" y2="42.164" width="0.2" layer="16"/>
+<wire x1="13.843" y1="42.164" x2="13.462" y2="41.783" width="0.2" layer="16"/>
+<wire x1="13.462" y1="41.783" x2="13.462" y2="36.703" width="0.2" layer="16"/>
+<wire x1="13.462" y1="36.703" x2="13.97" y2="36.195" width="0.2" layer="16"/>
+<wire x1="20.664" y1="36.198" x2="20.661" y2="36.195" width="0.2" layer="1"/>
+<wire x1="20.661" y1="36.195" x2="19.177" y2="36.195" width="0.2" layer="1"/>
+<via x="19.177" y="36.195" extent="1-16" drill="0.3"/>
+<wire x1="13.97" y1="36.195" x2="19.177" y2="36.195" width="0.2" layer="16"/>
 </signal>
 <signal name="19">
@@
 <wire x1="18.288" y1="44.196" x2="17.740484375" y2="44.743515625" width="0.2" layer="16"/>
 </signal>
-<signal name="N$17">
-<contactref element="U$1" pad="1"/>
-<contactref element="R1" pad="2"/>
-<wire x1="15.6938875" y1="43.561" x2="15.6972" y2="43.5576875" width="0.2" layer="16"/>
-<wire x1="15.6972" y1="43.5576875" x2="15.6972" y2="42.164" width="0.2" layer="16"/>
-</signal>
 </signals>
