File: RF-BM-2652P2/cc2652p_rf-star.brd (EAGLE design)
At the start: 25.3 x 57.3 mm, 44 parts, among them IC2 CP2102, J3 CORTEX_DEBUG_SMD, J5 TYPE-C-31-M-12, Q1 SI2323DS, U1 MCP73831, U2 ap2112k-3.3, U3 XC61CN3202MR-G

Commit message: Add files via upload
Parts:
- added C13: 220uF, Capacitor:CAPM7343X310
- added Q2: SI2323DS, SI2323DS:SOT23
- added R17, R18: 100k, RC0402FR-073M6L:RESC1005X40N
- added SJ1: PSM, pimoroni-misc:SMALL_SOLDER_JUMPER_CLOSED
- added U4: MMDT2907A-7-F, MMDT2907A-7-F:SOT65P210X110-6N
- moved BTN1 3.81 mm to (20.0, 23.6)
- moved BTN2 3.81 mm to (16.2, 23.6)
- moved C3 2.29 mm to (9.40, 45.8)
- moved R1 2.29 mm to (15.3, 45.8)
- moved R16 2.29 mm to (15.2, 47.0)
- moved U$1 2.29 mm to (12.3, 43.2)
- moved R15 2.29 mm to (8.52, 47.0)
- moved IC2 0.63 mm to (10.2, 14.7)
Connections:
- new net N$10: R18.2, U4.2, U4.3, U4.5
- new net N$13: Q2.1, R17.2, U4.6
- new net V+: C2.1, C4.1, IC2.6, IC2.7, Q2.3, R9.1, SJ1.1, U2.5, U4.4
- net +3V3: now also C13.1, Q2.2, SJ1.2, U4.1; no longer C2.1, C4.1, IC2.6, IC2.7, R9.1, U2.5
- net GND: now also C13.2, J3.9, R17.1, R18.1; no longer J3.3, J3.5
Routing:
- net V+: track 0.00 -> 41.9 mm, vias 0 -> 2
- net N$13: track 0.00 -> 9.69 mm, vias 0 -> 2
- net N$10: track 0.00 -> 6.93 mm
- net 15: track 42.2 -> 48.5 mm, vias 2 -> 3
- net +3V3: track 104.0 -> 109.6 mm, vias 3 -> 1
- net 14: track 18.2 -> 21.6 mm
- net 10: track 10.1 -> 12.7 mm
- net 20: track 23.7 -> 25.3 mm
- net GND: track 17.1 -> 18.1 mm, vias 81 -> 82
- net +5V: track 55.0 -> 55.8 mm
- net TDI: track 35.3 -> 36.1 mm
- net TDO: track 30.4 -> 29.6 mm
- net RTS: track 5.84 -> 5.15 mm
- net 13: track 34.4 -> 33.8 mm
- net 8: track 18.6 -> 19.2 mm
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Other:
- board text added: "DIO16/TDO"
- board text added: "DIO17/TDI"
