File: RF-BM-2652P2/cc2652p_rf-star.sch (EAGLE design)
At the start: 41 parts, among them IC2 CP2102, J3 CORTEX_DEBUG_SMD, J5 TYPE-C-31-M-12, Q1 SI2323DS, U1 MCP73831, U2 ap2112k-3.3, U3 XC61CN3202MR-G

Commit message: Add files via upload
Connections:
- net RES: now also J3.!RESET
Changed lines of the file:
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@@
 <label x="91.44" y="43.18" size="1.778" layer="95"/>
+</segment>
+<segment>
+<pinref part="J3" gate="G$1" pin="!RESET"/>
+<wire x1="195.58" y1="50.8" x2="203.2" y2="50.8" width="0.1524" layer="91"/>
+<label x="198.12" y="50.8" size="1.778" layer="95"/>
 </segment>
 </net>

Commit message: Add files via upload
RX TX fix
Connections:
- removed net DIO_12: IC2.TXD
- removed net DIO_13: IC2.RXD
- net 12: now also IC2.TXD
- net 13: now also IC2.RXD
Changed lines of the file:
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@@
-</segment>
-</net>
-<net name="DIO_12" class="0">
-<segment>
-<pinref part="IC2" gate="G$1" pin="TXD"/>
-<wire x1="66.04" y1="127" x2="76.2" y2="127" width="0.1524" layer="91"/>
-<label x="68.58" y="127" size="1.778" layer="95"/>
 </segment>
 </net>
@@
 <wire x1="106.68" y1="58.42" x2="114.3" y2="58.42" width="0.1524" layer="91"/>
 <label x="109.22" y="58.42" size="1.778" layer="95"/>
-</segment>
-</net>
-<net name="DIO_13" class="0">
-<segment>
-<pinref part="IC2" gate="G$1" pin="RXD"/>
-<wire x1="66.04" y1="124.46" x2="76.2" y2="124.46" width="0.1524" layer="91"/>
-<label x="68.58" y="124.46" size="1.778" layer="95"/>
 </segment>
 </net>
@@
 <label x="109.22" y="71.12" size="1.778" layer="95"/>
 </segment>
+<segment>
+<pinref part="IC2" gate="G$1" pin="RXD"/>
+<wire x1="66.04" y1="124.46" x2="76.2" y2="124.46" width="0.1524" layer="91"/>
+<label x="73.66" y="124.46" size="1.778" layer="95"/>
+</segment>
 </net>
 <net name="12" class="0">
@@
 <label x="109.22" y="73.66" size="1.778" layer="95"/>
 </segment>
-</net>
+<segment>
+<pinref part="IC2" gate="G$1" pin="TXD"/>
+<wire x1="66.04" y1="127" x2="76.2" y2="127" width="0.1524" layer="91"/>
+<label x="73.66" y="127" size="1.778" layer="95"/>
+</segment>
+</net>

Commit message: Add files via upload
Parts:
- removed C3: 0.1uF, SparkFun-Capacitors:0.1UF-0603-25V-(+80/-20%)
- removed R1: 100k, RC0402FR-073M6L:RC0402FR-073M6L
Connections:
- removed net N$4: C4.1, IC2.VDD, R9.1
- net +3V3: now also C4.1, IC2.REGIN, IC2.VDD, R9.1; no longer R1.1
- net +5V: no longer IC2.REGIN
- net GND: no longer C3.2
- net RES: no longer C3.1, R1.2
Changed lines of the file:
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@@
 <part name="C1" library="SparkFun-Capacitors" library_urn="urn:adsk.eagle:library:510" deviceset="10UF" device="-0603-6.3V-20%" package3d_urn="urn:adsk.eagle:package:37414/1" value="10uF"/>
 <part name="C2" library="SparkFun-Capacitors" library_urn="urn:adsk.eagle:library:510" deviceset="10UF" device="-0603-6.3V-20%" package3d_urn="urn:adsk.eagle:package:37414/1" value="10uF"/>
-<part name="R1" library="RC0402FR-073M6L" deviceset="RC0402FR-073M6L" device="" value="100k"/>
-<part name="C3" library="SparkFun-Capacitors" deviceset="0.1UF" device="-0603-25V-(+80/-20%)" package3d_urn="urn:adsk.eagle:package:37414/1" value="0.1uF"/>
-<part name="GND8" library="supply1" library_urn="urn:adsk.eagle:library:371" deviceset="GND" device=""/>
 <part name="GND10" library="supply1" library_urn="urn:adsk.eagle:library:371" deviceset="GND" device=""/>
 <part name="GND11" library="supply1" library_urn="urn:adsk.eagle:library:371" deviceset="GND" device=""/>
@@
 <part name="R12" library="RC0402FR-073M6L" deviceset="RC0402FR-073M6L" device="" value="2.2k"/>
 <part name="D6" library="SparkFun-LED" library_urn="urn:adsk.eagle:library:529" deviceset="LED-BLUE" device="0603" package3d_urn="urn:adsk.eagle:package:39354/1" value="BLUE"/>
-<part name="P+5" library="supply1" library_urn="urn:adsk.eagle:library:371" deviceset="+5V" device=""/>
 <part name="P+6" library="supply1" library_urn="urn:adsk.eagle:library:371" deviceset="+5V" device=""/>
 <part name="J3" library="SparkFun-Connectors" library_urn="urn:adsk.eagle:library:513" deviceset="CORTEX_DEBUG" device="_SMD" package3d_urn="urn:adsk.eagle:package:38289/1"/>
@@
 <part name="GND3" library="supply1" library_urn="urn:adsk.eagle:library:371" deviceset="GND" device=""/>
 <part name="GND9" library="supply1" library_urn="urn:adsk.eagle:library:371" deviceset="GND" device=""/>
+<part name="P+5" library="supply1" library_urn="urn:adsk.eagle:library:371" deviceset="+5V" device=""/>
+<part name="+3V2" library="supply1" library_urn="urn:adsk.eagle:library:371" deviceset="+3V3" device=""/>
 </parts>
 <sheets>
@@
 <attribute name="VALUE" x="148.844" y="190.881" size="1.778" layer="96" font="vector"/>
 </instance>
-<instance part="R1" gate="G$1" x="111.76" y="43.18" smashed="yes" rot="R180">
-<attribute name="NAME" x="111.76" y="41.656" size="1.778" layer="95" font="vector" rot="R180" align="bottom-center"/>
-</instance>
-<instance part="C3" gate="G$1" x="99.06" y="25.4" smashed="yes">
-<attribute name="NAME" x="100.584" y="28.321" size="1.778" layer="95" font="vector"/>
-<attribute name="VALUE" x="100.584" y="23.241" size="1.778" layer="96" font="vector"/>
-</instance>
-<instance part="GND8" gate="1" x="99.06" y="17.78" smashed="yes">
-<attribute name="VALUE" x="96.52" y="15.24" size="1.778" layer="96"/>
-</instance>
 <instance part="GND10" gate="1" x="205.74" y="76.2" smashed="yes">
 <attribute name="VALUE" x="203.2" y="73.66" size="1.778" layer="96"/>
@@
 <attribute name="VALUE" x="175.895" y="182.372" size="1.778" layer="96" font="vector" rot="R270" align="top-left"/>
 </instance>
-<instance part="P+5" gate="1" x="20.32" y="157.48" smashed="yes">
-<attribute name="VALUE" x="17.78" y="152.4" size="1.778" layer="96" rot="R90"/>
-</instance>
 <instance part="P+6" gate="1" x="93.98" y="149.86" smashed="yes" rot="R270">
 <attribute name="VALUE" x="88.9" y="152.4" size="1.778" layer="96"/>
@@
 <instance part="GND9" gate="1" x="137.16" y="48.26" smashed="yes">
 <attribute name="VALUE" x="134.62" y="45.72" size="1.778" layer="96"/>
+</instance>
+<instance part="P+5" gate="1" x="22.86" y="147.32" smashed="yes" rot="R90">
+<attribute name="VALUE" x="27.94" y="144.78" size="1.778" layer="96" rot="R180"/>
+</instance>
+<instance part="+3V2" gate="G$1" x="17.78" y="157.48" smashed="yes">
+<attribute name="VALUE" x="15.24" y="152.4" size="1.778" layer="96" rot="R90"/>
 </instance>
 </instances>
@@
 <pinref part="C2" gate="G$1" pin="2"/>
 <wire x1="147.32" y1="190.5" x2="147.32" y2="185.42" width="0.1524" layer="91"/>
-</segment>
-<segment>
-<pinref part="C3" gate="G$1" pin="2"/>
-<wire x1="99.06" y1="22.86" x2="99.06" y2="20.32" width="0.1524" layer="91"/>
-<pinref part="GND8" gate="1" pin="GND"/>
 </segment>
 <segment>
@@
 </segment>
 </net>
-<net name="N$4" class="0">
-<segment>
-<pinref part="C4" gate="G$1" pin="1"/>
-<pinref part="R9" gate="G$1" pin="1"/>
-<wire x1="10.16" y1="144.78" x2="10.16" y2="142.24" width="0.1524" layer="91"/>
-<pinref part="IC2" gate="G$1" pin="VDD"/>
-<wire x1="10.16" y1="142.24" x2="27.94" y2="142.24" width="0.1524" layer="91"/>
-<junction x="10.16" y="142.24"/>
-</segment>
-</net>
 <net name="N$7" class="0">
 <segment>
@@
 </segment>
 <segment>
-<pinref part="IC2" gate="G$1" pin="VBUS"/>
-<wire x1="27.94" y1="147.32" x2="20.32" y2="147.32" width="0.1524" layer="91"/>
-<pinref part="IC2" gate="G$1" pin="REGIN"/>
-<wire x1="20.32" y1="147.32" x2="20.32" y2="149.86" width="0.1524" layer="91"/>
-<wire x1="20.32" y1="149.86" x2="27.94" y2="149.86" width="0.1524" layer="91"/>
-<wire x1="20.32" y1="149.86" x2="20.32" y2="154.94" width="0.1524" layer="91"/>
-<junction x="20.32" y="149.86"/>
-<pinref part="P+5" gate="1" pin="+5V"/>
-</segment>
-<segment>
 <pinref part="R8" gate="G$1" pin="2"/>
 <wire x1="88.9" y1="149.86" x2="91.44" y2="149.86" width="0.1524" layer="91"/>
@@
 <wire x1="106.68" y1="53.34" x2="114.3" y2="53.34" width="0.1524" layer="91"/>
 <pinref part="P+8" gate="1" pin="+5V"/>
+</segment>
+<segment>
+<pinref part="IC2" gate="G$1" pin="VBUS"/>
+<wire x1="27.94" y1="147.32" x2="25.4" y2="147.32" width="0.1524" layer="91"/>
+<pinref part="P+5" gate="1" pin="+5V"/>
 </segment>
 </net>
@@
 </segment>
 <segment>
-<pinref part="R1" gate="G$1" pin="1"/>
-<wire x1="121.92" y1="43.18" x2="129.54" y2="43.18" width="0.1524" layer="91"/>
-<label x="124.46" y="43.18" size="1.778" layer="95"/>
-</segment>
-<segment>
 <pinref part="J3" gate="G$1" pin="VCC"/>
 <wire x1="162.56" y1="60.96" x2="154.94" y2="60.96" width="0.1524" layer="91"/>
@@
 <wire x1="129.54" y1="60.96" x2="137.16" y2="60.96" width="0.1524" layer="91"/>
 <label x="129.54" y="60.96" size="1.778" layer="95"/>
+</segment>
+<segment>
+<pinref part="C4" gate="G$1" pin="1"/>
+<pinref part="R9" gate="G$1" pin="1"/>
+<wire x1="10.16" y1="144.78" x2="10.16" y2="142.24" width="0.1524" layer="91"/>
+<pinref part="IC2" gate="G$1" pin="VDD"/>
+<wire x1="10.16" y1="142.24" x2="17.78" y2="142.24" width="0.1524" layer="91"/>
+<junction x="10.16" y="142.24"/>
+<pinref part="IC2" gate="G$1" pin="REGIN"/>
+<wire x1="17.78" y1="142.24" x2="27.94" y2="142.24" width="0.1524" layer="91"/>
+<wire x1="17.78" y1="142.24" x2="17.78" y2="149.86" width="0.1524" layer="91"/>
+<wire x1="17.78" y1="149.86" x2="27.94" y2="149.86" width="0.1524" layer="91"/>
+<junction x="17.78" y="142.24"/>
+<wire x1="17.78" y1="149.86" x2="17.78" y2="154.94" width="0.1524" layer="91"/>
+<junction x="17.78" y="149.86"/>
+<pinref part="+3V2" gate="G$1" pin="+3V3"/>
 </segment>
 </net>
@@
 </segment>
 <segment>
-<pinref part="C3" gate="G$1" pin="1"/>
-<wire x1="99.06" y1="30.48" x2="99.06" y2="43.18" width="0.1524" layer="91"/>
-<pinref part="R1" gate="G$1" pin="2"/>
-<wire x1="99.06" y1="43.18" x2="101.6" y2="43.18" width="0.1524" layer="91"/>
-<wire x1="99.06" y1="43.18" x2="91.44" y2="43.18" width="0.1524" layer="91"/>
-<junction x="99.06" y="43.18"/>
-<label x="91.44" y="43.18" size="1.778" layer="95"/>
-</segment>
-<segment>

Commit message: Add files via upload
Parts:
- added C3: 100n, discretes-dev:CAP0402
- added R1: 2.2k, RC0402FR-073M6L:RC0402FR-073M6L
- added R15, R16: 0, RC0402FR-073M6L:RC0402FR-073M6L
- added U$1: MX25R8035FM1IL0, W25Q80BVSNIG:W25Q80BVSNIG
Connections:
- new net N$12: R15.2, U$1.HOLD/IO3
- new net N$15: R16.1, U$1.WP/IO2
- new net N$17: R1.2, U$1.CS
- net +3V3: now also C3.2, R1.1, R15.1, R16.2, U$1.VCC
- net 10: now also U$1.CLK
- net 8: now also U$1.DO/IO1
- net 9: now also U$1.DI/IO0
- net GND: now also C3.1, U$1.GND
Other:
- moved on the sheet: C1, C2, CN1, D5, D6, PAD1, PAD2, Q1, R11, R12, R13, R14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

Commit message: Add files via upload
Connections:
- removed net N$17: R1.2, U$1.CS
- net 20: now also R1.2, U$1.CS
Changed lines of the file:
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@@
 <label x="76.2" y="55.88" size="1.778" layer="95"/>
+</segment>
+<segment>
+<pinref part="U$1" gate="G$1" pin="CS"/>
+<pinref part="R1" gate="G$1" pin="2"/>
+<wire x1="269.24" y1="50.8" x2="276.86" y2="50.8" width="0.1524" layer="91"/>
+<label x="274.32" y="50.8" size="1.778" layer="95"/>
 </segment>
 </net>
@@
 </segment>
 </net>
-<net name="N$17" class="0">
-<segment>
-<pinref part="U$1" gate="G$1" pin="CS"/>
-<pinref part="R1" gate="G$1" pin="2"/>
-<wire x1="269.24" y1="50.8" x2="276.86" y2="50.8" width="0.1524" layer="91"/>
-</segment>
-</net>

Commit message: Add files via upload
Parts:
- added C13: 220uF, Capacitor:C_TANTALUM-2917(7343-METRIC)
- added Q2: SI2323DS, SI2323DS:SI2323DS
- added R17, R18: 100k, RC0402FR-073M6L:RC0402FR-073M6L
- added SJ1: PSM, pimoroni-misc:SMALL_SOLDER_JUMPER_CLOSED
- added U4: MMDT2907A-7-F, MMDT2907A-7-F:MMDT2907A-7-F
Connections:
- new net N$10: R18.2, U4.B1, U4.B2, U4.C1
- new net N$13: Q2.G, R17.2, U4.C2
- new net V+: C2.1, C4.1, IC2.REGIN, IC2.VDD, Q2.D, R9.1, SJ1.1, U2.OUT, U4.E1
- net +3V3: now also C13.1, Q2.S, SJ1.2, U4.E2; no longer C2.1, C4.1, IC2.REGIN, IC2.VDD, R9.1, U2.OUT
- net GND: now also C13.2, J3.GNDDTCT, R17.1, R18.1; no longer J3.GND@3, J3.GND@5
Other:
- moved on the sheet: CN1, D6, PAD1, PAD2, R11, R12, R2, U1, U3
